Commit message: First commit with simplify URDF

File: opendog_description/urdf/consts.xacro (robot description, xacro)
@@ -1,4 +1,5 @@
 <?xml version="1.0"?>
 <robot name="consts" xmlns:xacro="http://www.ros.org/wiki/xacro">
+    <xacro:property name="M_PI"  value="3.14159"/>
     <!-- joint limits -->
     <xacro:property name="hip_low_limit"  value="-1.57"/>
@@ -21,6 +22,15 @@
         <dynamics damping="0.01" friction="10000"/>
     </xacro:macro>
+    <xacro:property name="base_link_width" value="0.25"/>
+    <xacro:property name="base_link_height" value="0.28"/>
+    <xacro:property name="base_link_depth" value="0.875"/>
+    <xacro:property name="hip_link_length" value="0.20"/>
+    <xacro:property name="hip_link_radius" value="0.05"/>
+    <xacro:property name="uleg_link_radius" value="0.025"/>
+    <xacro:property name="lleg_link_radius" value="0.025"/>
+    <xacro:property name="uleg_link_length" value="0.20"/>
+    <xacro:property name="lleg_link_length" value="0.22"/>
     <!-- configure inertia -->
-    <xacro:property name="body_mass" value="3"/>
+    <xacro:property name="body_mass" value="50"/>
     <xacro:property name="body_inertia_x_len" value="0.28"/>
     <xacro:property name="body_inertia_y_len" value="0.172"/>

File: opendog_description/urdf/opendog_joints.xacro (robot description, xacro)
@@ -9,5 +9,5 @@
     <!-- *********  FR_hip joint ********* -->
     <joint name="FR_hip_joint" type="revolute">
-        <origin xyz="0.005372 -0.029025 0.34267" rpy="0 0 0"/>
+        <origin xyz="${base_link_depth/2} ${base_link_width/2} ${base_link_height/2}" rpy="0 0 0"/>
         <parent link="base_link"/>
         <child link="FR_hip_link"/>
@@ -17,5 +17,5 @@
     <!-- *********  FL_hip  ********* -->
     <joint name="FL_hip_joint" type="revolute">
-        <origin xyz="0.005091 -0.147198 0.340765" rpy="0 0 0"/>
+        <origin xyz="${base_link_depth/2} -${base_link_width/2} ${base_link_height/2}" rpy="0 0 0"/>
         <parent link="base_link"/>
         <child link="FL_hip_link"/>
@@ -25,5 +25,5 @@
     <!-- *********  BR_hip  ********* -->
     <joint name="BR_hip_joint" type="revolute">
-        <origin xyz="0.471531 -0.028918 0.340765" rpy="0 0 0"/>
+        <origin xyz="-${base_link_depth/2} ${base_link_width/2} ${base_link_height/2}" rpy="0 0 0"/>
         <parent link="base_link"/>
         <child link="BR_hip_link"/>
@@ -33,5 +33,5 @@
     <!-- *********  BL_hip  ********* -->
     <joint name="BL_hip_joint" type="revolute">
-        <origin xyz="0.471531 -0.147198 0.340765" rpy="0 0 0"/>
+        <origin xyz="-${base_link_depth/2} -${base_link_width/2} ${base_link_height/2}" rpy="0 0 0"/>
         <parent link="base_link"/>
         <child link="BL_hip_link"/>

File: opendog_description/urdf/opendog_links.xacro (robot description, xacro)
@@ -1,299 +1,326 @@
 <?xml version="1.0"?>
 <robot xmlns:xacro="http://www.ros.org/wiki/xacro">
-    <xacro:include filename="consts.xacro" />
-    <xacro:include filename="physics.xacro" />
-    <!-- load meshes -->
-    <xacro:macro name="body_mesh">
-        <mesh filename="file://$(find opendog_description)/meshes/body.stl" scale="0.001 0.001 0.001"/>
-    </xacro:macro>
-    <xacro:macro name="rightHip_mesh">
-        <mesh filename="file://$(find opendog_description)/meshes/RIGHT_HIP.stl" scale="0.001 0.001 0.001"/>
-    </xacro:macro>
-    <xacro:macro name="leftHip_mesh">
-        <mesh filename="file://$(find opendog_description)/meshes/LEFT_HIP.stl" scale="0.001 0.001 0.001"/>
-    </xacro:macro>
-    <xacro:macro name="rightUleg_mesh">
-        <mesh filename="file://$(find opendog_description)/meshes/RIGHT_ULEG.stl" scale="0.001 0.001 0.001"/>
-    </xacro:macro>
-    <xacro:macro name="leftUleg_mesh">
-        <mesh filename="file://$(find opendog_description)/meshes/LEFT_ULEG.stl" scale="0.001 0.001 0.001"/>
-    </xacro:macro>
-    <xacro:macro name="lleg_mesh">
-        <mesh filename="file://$(find opendog_description)/meshes/LLEG.stl" scale="0.001 0.001 0.001"/>
-    </xacro:macro>
-    <!-- *********** Inertial link *********** -->
-    <link name="world">
-    </link>
-    <!-- *********** base link *********** -->
-    <link name="base_link">
-        <inertial>
-          <origin xyz="0.2749797958231685 -0.08799492490648385 0.36444405374780864" rpy="0 0 0"/>
-          <mass value="5"/>
-          <inertia ixx="0.761631" iyy="4.077449" izz="3.905689" ixy="-0.001055" iyz="-0.000345" ixz="0.05479"/>
-        </inertial>
-        <visual>
-          <origin xyz="0 0 0" rpy="0 0 0"/>
-          <geometry>
-            <mesh filename="file://$(find opendog_description)/meshes/base_link.stl" scale="0.001 0.001 0.001"/>
-          </geometry>
-        </visual>
-        <collision>
-          <origin xyz="0 0 0" rpy="0 0 0"/>
-          <geometry>
-            <mesh filename="file://$(find opendog_description)/meshes/base_link.stl" scale="0.001 0.001 0.001"/>
-          </geometry>
-        </collision>
-    </link>
-    <!-- !!!!!!!!!!!!!!!!!!!!!!! HIPS !!!!!!!!!!!!!!!!!!!!!!!!!!!! -->
-    <!-- *********** FR_hip *********** -->
-    <link name="FR_hip_link">
-        <inertial>
-            <origin xyz="-0.09804953144426388 0.01537887460379041 0.00019055475909179886" rpy="0 0 0"/>
-            <mass value="2"/>
-            <inertia ixx="0.012708" iyy="0.026996" izz="0.026264" ixy="-0.000651" iyz="8.1e-05" ixz="-1.7e-05"/>
-        </inertial>
-        <visual>
-            <origin xyz="-0.005372 0.029025 -0.34267" rpy="0 0 0"/>
-            <geometry>
-              <mesh filename="file://$(find opendog_description)/meshes/FR_hip_link_2.stl" scale="0.001 0.001 0.001"/>
-            </geometry>
-        </visual>
-        <collision>
-            <origin xyz="-0.005372 0.029025 -0.34267" rpy="0 0 0"/>
-            <geometry>
-              <mesh filename="file://$(find opendog_description)/meshes/FR_hip_link_2.stl" scale="0.001 0.001 0.001"/>
-            </geometry>
-        </collision>
-    </link>
-    <!-- *********** FL_hip ********** -->
-    <link name="FL_hip_link">
-        <inertial>
-            <origin xyz="-0.09804956975710932 -0.015379348802188275 0.00019128110374050378" rpy="0 0 0"/>
-            <mass value="2"/>
-            <inertia ixx="0.012737" iyy="0.027034" izz="0.026319" ixy="0.000689" iyz="-4.8e-05" ixz="1.1e-05"/>
-        </inertial>
-        <visual>
-            <origin xyz="-0.005091 0.147198 -0.340765" rpy="0 0 0"/>
-            <geometry>
-              <mesh filename="file://$(find opendog_description)/meshes/FL_hip_link_2.stl" scale="0.001 0.001 0.001"/>
-            </geometry>
-        </visual>
-        <collision>
-            <origin xyz="-0.005091 0.147198 -0.340765" rpy="0 0 0"/>
-            <geometry>
-              <mesh filename="file://$(find opendog_description)/meshes/FL_hip_link_2.stl" scale="0.001 0.001 0.001"/>
-            </geometry>
-        </collision>
-    </link>
-    <!-- *********** BR_hip ********** -->
-    <link name="BR_hip_link">
-        <inertial>
-            <origin xyz="0.09804922989186687 0.015379343283856973 0.00019128110374272422" rpy="0 0 0"/>
-            <mass value="2"/>
-            <inertia ixx="0.012708" iyy="0.027002" izz="0.026258" ixy="0.000651" iyz="5e-05" ixz="-1e-05"/>
-        </inertial>
-        <visual>
-            <origin xyz="-0.471531 0.028918 -0.340765" rpy="0 0 0"/>
-            <geometry>
-              <mesh filename="file://$(find opendog_description)/meshes/BR_hip_link_2.stl" scale="0.001 0.001 0.001"/>
-            </geometry>
-        </visual>
-        <collision>
-            <origin xyz="-0.471531 0.028918 -0.340765" rpy="0 0 0"/>
-            <geometry>
-              <mesh filename="file://$(find opendog_description)/meshes/BR_hip_link_2.stl" scale="0.001 0.001 0.001"/>
-            </geometry>
-        </collision>
-    </link>
-    <!-- *********** BL_hip ********** -->
-    <link name="BL_hip_link">
-        <inertial>
-            <origin xyz="0.09804922228400342 -0.015379345578511366 0.00019128032686782648" rpy="0 0 0"/>
-            <mass value="2"/>
-            <inertia ixx="0.012784" iyy="0.027006" izz="0.026333" ixy="-0.000657" iyz="-4.9e-05" ixz="-1.1e-05"/>
-        </inertial>
-        <visual>
-            <origin xyz="-0.471531 0.147198 -0.340765" rpy="0 0 0"/>
-            <geometry>
-              <mesh filename="file://$(find opendog_description)/meshes/BL_hip_link_2.stl" scale="0.001 0.001 0.001"/>
-            </geometry>
-        </visual>
-        <collision>
-            <origin xyz="-0.471531 0.147198 -0.340765" rpy="0 0 0"/>
-            <geometry>
-              <mesh filename="file://$(find opendog_description)/meshes/BL_hip_link_2.stl" scale="0.001 0.001 0.001"/>
-            </geometry>
-        </collision>
-    </link>
-    <!-- !!!!!!!!!!!!!!!!!!!!!!! ULEGs !!!!!!!!!!!!!!!!!!!!!!!!!!!! -->
-    <!-- *********** FR_uleg ********** -->
-    <link name="FR_uleg_link">
-        <inertial>
-            <origin xyz="0.024785646151847765 0.06031237152858331 -0.02501775170684245" rpy="0 0 0"/>
-            <mass value="2.7"/>
-            <inertia ixx="0.060385" iyy="0.086191" izz="0.061956" ixy="0.004251" iyz="-0.003909" ixz="0.027901"/>
-        </inertial>
-        <visual>
-            <origin xyz="0.094268 -0.037335 -0.34267" rpy="0 0 0"/>
-            <geometry>
-              <mesh filename="file://$(find opendog_description)/meshes/FR_uleg_link_2.stl" scale="0.001 0.001 0.001"/>
-            </geometry>
-        </visual>
-        <collision>
-            <origin xyz="0.094268 -0.037335 -0.34267" rpy="0 0 0"/>
-            <geometry>
-              <mesh filename="file://$(find opendog_description)/meshes/FR_uleg_link_2.stl" scale="0.001 0.001 0.001"/>
-            </geometry>
-        </collision>
-    </link>
-    <!-- *********** FL_uleg ********** -->
-    <link name="FL_uleg_link">
-        <inertial>
-            <origin xyz="0.02578305194465416 -0.06037459079064242 -0.02602287407328735" rpy="0 0 0"/>
-            <mass value="2.7"/>
-            <inertia ixx="0.051391" iyy="0.085806" izz="0.071334" ixy="-0.006201" iyz="0.003973" ixz="0.025851"/>
-        </inertial>
-        <visual>
-            <origin xyz="0.094549 0.213558 -0.340765" rpy="0 0 0"/>
-            <geometry>
-              <mesh filename="file://$(find opendog_description)/meshes/FL_uleg_link_2.stl" scale="0.001 0.001 0.001"/>
-            </geometry>
-        </visual>
-        <collision>
-            <origin xyz="0.094549 0.213558 -0.340765" rpy="0 0 0"/>
-            <geometry>
-              <mesh filename="file://$(find opendog_description)/meshes/FL_uleg_link_2.stl" scale="0.001 0.001 0.001"/>
-            </geometry>
-        </collision>
-    </link>
-    <!-- *********** BR_uleg ********** -->
-    <link name="BR_uleg_link">
-        <inertial>
-            <origin xyz="-0.02478596816754486 0.060312838896795826 -0.025017037989093105" rpy="0 0 0"/>
-            <mass value="2.7"/>
-            <inertia ixx="0.061911" iyy="0.085831" izz="0.060788" ixy="-0.005251" iyz="-0.005031" ixz="-0.027715"/>
-        </inertial>
-        <visual>
-            <origin xyz="-0.571171 -0.037442 -0.340765" rpy="0 0 0"/>
-            <geometry>
-              <mesh filename="file://$(find opendog_description)/meshes/BR_uleg_link_2.stl" scale="0.001 0.001 0.001"/>
-            </geometry>
-        </visual>
-        <collision>
-            <origin xyz="-0.571171 -0.037442 -0.340765" rpy="0 0 0"/>
-            <geometry>
-              <mesh filename="file://$(find opendog_description)/meshes/BR_uleg_link_2.stl" scale="0.001 0.001 0.001"/>
-            </geometry>
-        </collision>
-    </link>
-    <!-- *********** BL_uleg ********** -->
-    <link name="BL_uleg_link">
-        <inertial>
-            <origin xyz="-0.024912930584652382 -0.06035054910971113 -0.02514445341334004" rpy="0 0 0"/>
-            <mass value="2.7"/>
-            <inertia ixx="0.061226" iyy="0.085803" izz="0.061502" ixy="0.005391" iyz="0.005035" ixz="-0.027705"/>
-        </inertial>
-        <visual>
-            <origin xyz="-0.571171 0.213558 -0.340765" rpy="0 0 0"/>
-            <geometry>
-              <mesh filename="file://$(find opendog_description)/meshes/BL_uleg_link_2.stl" scale="0.001 0.001 0.001"/>
-            </geometry>
-        </visual>
-        <collision>
-            <origin xyz="-0.571171 0.213558 -0.340765" rpy="0 0 0"/>
-            <geometry>
-              <mesh filename="file://$(find opendog_description)/meshes/BL_uleg_link_2.stl" scale="0.001 0.001 0.001"/>
-            </geometry>
-        </collision>
-    </link>
-    <!-- !!!!!!!!!!!!!!!!!!!!!!! LLEGs !!!!!!!!!!!!!!!!!!!!!!!!!!!! -->
-    <!-- *********** FR_lleg ********** -->
-    <link name="FR_lleg_link">
-        <inertial>
-            <origin xyz="-0.06309907279078683 -0.04027150228827056 -0.06310352710956241" rpy="0 0 0"/>
-            <mass value="0.3"/>
-            <inertia ixx="0.007726" iyy="0.021253" izz="0.015039" ixy="0.000248" iyz="0.00018" ixz="-0.008798"/>
-        </inertial>
-        <visual>
-            <origin xyz="-0.0467 -0.119335 -0.201701" rpy="0 0 0"/>
-            <geometry>
-              <mesh filename="file://$(find opendog_description)/meshes/FR_lleg_link_2.stl" scale="0.001 0.001 0.001"/>
-            </geometry>
-        </visual>
-        <collision>
-            <origin xyz="-0.0467 -0.119335 -0.201701" rpy="0 0 0"/>
-            <geometry>
-              <mesh filename="file://$(find opendog_description)/meshes/FR_lleg_link_2.stl" scale="0.001 0.001 0.001"/>
-            </geometry>
-        </collision>
-    </link>
-    <!-- *********** FL_lleg ********** -->
-    <link name="FL_lleg_link">
-        <inertial>
-            <origin xyz="-0.06309910896868268 0.04027103185737707 -0.06310379848106407" rpy="0 0 0"/>
-            <mass value="0.3"/>
-            <inertia ixx="0.010996" iyy="0.029242" izz="0.019764" ixy="0.000158" iyz="0.000113" ixz="-0.012783"/>
-        </inertial>
-        <visual>
-            <origin xyz="-0.046419 0.295558 -0.199797" rpy="0 0 0"/>
-            <geometry>
-              <mesh filename="file://$(find opendog_description)/meshes/FL_lleg_link_2.stl" scale="0.001 0.001 0.001"/>
-            </geometry>
-        </visual>
-        <collision>
-            <origin xyz="-0.046419 0.295558 -0.199797" rpy="0 0 0"/>
-            <geometry>
-              <mesh filename="file://$(find opendog_description)/meshes/FL_lleg_link_2.stl" scale="0.001 0.001 0.001"/>
-            </geometry>
-        </collision>
-    </link>
-      <!-- *********** BR_lleg ********** -->
-    <link name="BR_lleg_link">
-        <inertial>
-            <origin xyz="0.06309976910343829 -0.04027103737571108 -0.06310379848106251" rpy="0 0 0"/>
-            <mass value="0.3"/>
-            <inertia ixx="0.006577" iyy="0.021257" izz="0.016183" ixy="0.00012" iyz="-6.8e-05" ixz="0.00823"/>
-        </inertial>
-        <visual>
-            <origin xyz="-0.430202 -0.119442 -0.199797" rpy="0 0 0"/>
-            <geometry>
-              <mesh filename="file://$(find opendog_description)/meshes/BR_lleg_link_2.stl" scale="0.001 0.001 0.001"/>
-            </geometry>
-        </visual>
-        <collision>
-            <origin xyz="-0.430202 -0.119442 -0.199797" rpy="0 0 0"/>
-            <geometry>
-              <mesh filename="file://$(find opendog_description)/meshes/BR_lleg_link_2.stl" scale="0.001 0.001 0.001"/>
-            </geometry>
-        </collision>
-    </link>
-    <!-- *********** BL_lleg ********** -->
-    <link name="BL_lleg_link">
-        <inertial>
-            <origin xyz="0.06309976363052966 0.040271031313545036 -0.06310380154178746" rpy="0 0 0"/>
-            <mass value="0.3"/>
-            <inertia ixx="0.006615" iyy="0.021256" izz="0.016145" ixy="-0.000143" iyz="8.3e-05" ixz="0.008252"/>
-        </inertial>
-        <visual>
-            <origin xyz="-0.430202 0.295558 -0.199797" rpy="0 0 0"/>
-            <geometry>
-              <mesh filename="file://$(find opendog_description)/meshes/BL_lleg_link_2.stl" scale="0.001 0.001 0.001"/>
-            </geometry>
-        </visual>
-        <collision>
-            <origin xyz="-0.430202 0.295558 -0.199797" rpy="0 0 0"/>
-            <geometry>
-              <mesh filename="file://$(find opendog_description)/meshes/BL_lleg_link_2.stl" scale="0.001 0.001 0.001"/>
-            </geometry>
-            <surface>
-                <friction>
-                    <ode>
-                        <mu>1</mu>
-                        <mu2>1</mu2>
-                        <fdir1>1 0 0</fdir1>
-                    </ode>
-                </friction>
-            </surface>
-        </collision>
-    </link>
+  <xacro:include filename="consts.xacro" />
+  <xacro:include filename="physics.xacro" />
+  <!-- load meshes -->
+  <xacro:macro name="body_mesh">
+    <mesh filename="file://$(find opendog_description)/meshes/body.stl" scale="0.001 0.001 0.001"/>
+  </xacro:macro>
+  <xacro:macro name="rightHip_mesh">
+    <mesh filename="file://$(find opendog_description)/meshes/RIGHT_HIP.stl" scale="0.001 0.001 0.001"/>
+  </xacro:macro>
+  <xacro:macro name="leftHip_mesh">
+    <mesh filename="file://$(find opendog_description)/meshes/LEFT_HIP.stl" scale="0.001 0.001 0.001"/>
+  </xacro:macro>
+  <xacro:macro name="rightUleg_mesh">
+    <mesh filename="file://$(find opendog_description)/meshes/RIGHT_ULEG.stl" scale="0.001 0.001 0.001"/>
+  </xacro:macro>
+  <xacro:macro name="leftUleg_mesh">
+    <mesh filename="file://$(find opendog_description)/meshes/LEFT_ULEG.stl" scale="0.001 0.001 0.001"/>
+  </xacro:macro>
+  <xacro:macro name="lleg_mesh">
+    <mesh filename="file://$(find opendog_description)/meshes/LLEG.stl" scale="0.001 0.001 0.001"/>
+  </xacro:macro>
+  <!-- *********** Inertial link *********** -->
+  <link name="world">
+  </link>
+  <!-- *********** base link *********** -->
+  <link name="base_link">
+    <inertial>
+      <origin xyz="0 0 ${base_link_height/2}" rpy="0 ${M_PI/2} 0"/>
+      <mass value="${body_mass}"/>
+      <inertia ixx="${(1/12) * body_mass * (base_link_depth * base_link_depth + base_link_width * base_link_width ) }" iyy="${(1/12) * body_mass * (base_link_depth * base_link_depth + base_link_height * base_link_height ) }" izz="${(1/12) * body_mass * (base_link_width * base_link_width + base_link_height * base_link_height ) }" ixy="0.0" iyz="0.0" ixz="0.0"/>
+    </inertial>
+    <visual>
+      <origin xyz="0 0 ${base_link_height/2}" rpy="0 0 0"/>
+      <geometry>
+        <box size="${base_link_depth} ${base_link_width} ${base_link_height}"/>
+      </geometry>
+    </visual>
+    <collision>
+      <origin xyz="0 0 ${base_link_height/2}" rpy="0 0 0"/>
+      <geometry>
+        <box size="${base_link_depth} ${base_link_width} ${base_link_height}"/>
+      </geometry>
+    </collision>
+  </link>
+  <!-- !!!!!!!!!!!!!!!!!!!!!!! HIPS !!!!!!!!!!!!!!!!!!!!!!!!!!!! -->
+  <!-- *********** FR_hip *********** -->
+  <link name="FR_hip_link">
+    <inertial>
+      <origin xyz="0.0 0.0 0.0" rpy="${M_PI/2} ${M_PI/2} 0"/>
+      <mass value="${hip_mass}"/>
+      <inertia ixx="${(1/12) * hip_mass * (3 * hip_link_radius * hip_link_radius + hip_link_length * hip_link_length) }"
+                iyy="${(1/12) * hip_mass * (3 * hip_link_radius * hip_link_radius) }"
+                izz="${(1/12) * hip_mass * (3 * hip_link_radius * hip_link_radius + hip_link_length * hip_link_length) }"
+                ixy="0.0" iyz="0.0" ixz="0.0"/>
+    </inertial>
+    <visual>
+      <origin xyz="0.0 0.0 0.0" rpy="0 ${M_PI/2} 0"/>
+      <geometry>
+        <cylinder radius="${hip_link_radius}" length="${hip_link_length}"/>
+      </geometry>
+    </visual>
+    <collision>
+      <origin xyz="0.0 0.0 0.0" rpy="0 ${M_PI/2}  0"/>
+      <geometry>
+        <cylinder radius="${hip_link_radius}" length="${hip_link_length}"/>
+      </geometry>
+    </collision>
+  </link>
+  <!-- *********** FL_hip ********** -->
+  <link name="FL_hip_link">
+    <inertial>
+      <origin xyz="0.0 0.0 0.0" rpy="${M_PI/2} ${M_PI/2} 0"/>
+      <mass value="${hip_mass}"/>
+      <inertia ixx="${(1/12) * hip_mass * (3 * hip_link_radius * hip_link_radius + hip_link_length * hip_link_length) }"
+                iyy="${(1/12) * hip_mass * (3 * hip_link_radius * hip_link_radius) }"
+                izz="${(1/12) * hip_mass * (3 * hip_link_radius * hip_link_radius + hip_link_length * hip_link_length) }"
+                ixy="0.0" iyz="0.0" ixz="0.0"/>
+    </inertial>
+    <visual>
+      <origin xyz="0.0 0.0 0.0" rpy="0 ${M_PI/2} 0"/>
+      <geometry>
+        <cylinder radius="${hip_link_radius}" length="${hip_link_length}"/>
+      </geometry>
+    </visual>
+    <collision>
+      <origin xyz="0.0 0.0 0.0" rpy="0 ${M_PI/2}  0"/>
+      <geometry>
+        <cylinder radius="${hip_link_radius}" length="${hip_link_length}"/>
+      </geometry>
+    </collision>
+  </link>
+  <!-- *********** BR_hip ********** -->
+  <link name="BR_hip_link">
+    <inertial>
+      <origin xyz="0.0 0.0 0.0" rpy="${M_PI/2} ${M_PI/2} 0"/>
+      <mass value="${hip_mass}"/>
+      <inertia ixx="${(1/12) * hip_mass * (3 * hip_link_radius * hip_link_radius + hip_link_length * hip_link_length) }"
+                iyy="${(1/12) * hip_mass * (3 * hip_link_radius * hip_link_radius) }"
+                izz="${(1/12) * hip_mass * (3 * hip_link_radius * hip_link_radius + hip_link_length * hip_link_length) }"
+                ixy="0.0" iyz="0.0" ixz="0.0"/>
+    </inertial>
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