Commit message: Updated the opendog_description: launch, urdf, meshes.

File: opendog_description/urdf/opendog_joints.xacro (robot description, xacro)
@@ -19,9 +19,9 @@
     <!-- *********  FR_hip joint ********* -->
     <joint name="FR_hip_joint" type="revolute">
-        <axis xyz="1.0 -0.0 0.0"/>
-        <origin xyz="0.120789 -0.018307 0.263166" rpy="0 0 0"/>
+        <origin xyz="0.005372 -0.029025 0.34267" rpy="0 0 0"/>
         <parent link="base_link"/>
         <child link="FR_hip_link"/>
-        <limit upper="0.349066" lower="-0.349066" effort="100" velocity="100"/>
+        <axis xyz="1.0 -0.0 0.0"/>
+  <limit upper="0.174533" lower="-0.174533" effort="100" velocity="100"/>
         <xacro:if value="${use_dynamics}">
             <xacro:hip_joint_dynamics></xacro:hip_joint_dynamics>
@@ -30,9 +30,9 @@
     <!-- *********  FL_hip  ********* -->
     <joint name="FL_hip_joint" type="revolute">
-        <axis xyz="-1.0 0.0 -0.0"/>
-        <origin xyz="0.120789 -0.136588 0.263166" rpy="0 0 0"/>
+        <origin xyz="0.005091 -0.147198 0.340765" rpy="0 0 0"/>
         <parent link="base_link"/>
         <child link="FL_hip_link"/>
-        <limit upper="0.349066" lower="-0.785398" effort="100" velocity="100"/>
+        <axis xyz="-1.0 0.0 -0.0"/>
+        <limit upper="0.174533" lower="-0.174533" effort="100" velocity="100"/>
         <xacro:if value="${use_dynamics}">
             <xacro:hip_joint_dynamics></xacro:hip_joint_dynamics>
@@ -41,9 +41,9 @@
     <!-- *********  BR_hip  ********* -->
     <joint name="BR_hip_joint" type="revolute">
-        <axis xyz="1.0 -0.0 -0.0"/>
-        <origin xyz="0.468789 -0.018307 0.263166" rpy="0 0 0"/>
+        <origin xyz="0.471531 -0.028918 0.340765" rpy="0 0 0"/>
         <parent link="base_link"/>
         <child link="BR_hip_link"/>
-        <limit upper="0.349066" lower="-0.785398" effort="100" velocity="100"/>
+        <axis xyz="1.0 -0.0 -0.0"/>
+        <limit upper="0.174533" lower="-0.174533" effort="100" velocity="100"/>
         <xacro:if value="${use_dynamics}">
             <xacro:hip_joint_dynamics></xacro:hip_joint_dynamics>
@@ -52,9 +52,9 @@
     <!-- *********  BL_hip  ********* -->
     <joint name="BL_hip_joint" type="revolute">
-        <axis xyz="-1.0 0.0 0.0"/>
-        <origin xyz="0.468789 -0.136588 0.263166" rpy="0 0 0"/>
+        <origin xyz="0.471531 -0.147198 0.340765" rpy="0 0 0"/>
         <parent link="base_link"/>
         <child link="BL_hip_link"/>
-        <limit upper="0.436332" lower="-0.785398" effort="100" velocity="100"/>
+        <axis xyz="-1.0 0.0 0.0"/>
+        <limit upper="0.174533" lower="-0.174533" effort="100" velocity="100"/>
         <xacro:if value="${use_dynamics}">
             <xacro:hip_joint_dynamics></xacro:hip_joint_dynamics>
@@ -63,9 +63,9 @@
     <!-- *********  FR_uleg joint ********* -->
     <joint name="FR_uleg_joint" type="revolute">
-        <axis xyz="-0.0 -0.999043 -0.043739"/>
-        <origin xyz="-0.09964 0.066296 0.002902" rpy="0 0 0"/>
+        <origin xyz="-0.09964 0.06636 0.0" rpy="0 0 0"/>
         <parent link="FR_hip_link"/>
         <child link="FR_uleg_link"/>
-        <xacro:uleg_limits></xacro:uleg_limits>
+        <axis xyz="-0.0 -1.0 0.0"/>
+        <limit upper="0.785398" lower="-2.356194" effort="100" velocity="100"/>
         <xacro:if value="${use_dynamics}">
             <xacro:uleg_joint_dynamics></xacro:uleg_joint_dynamics>
@@ -74,9 +74,9 @@
     <!-- *********  FL_uleg  ********* -->
     <joint name="FL_uleg_joint" type="revolute">
-        <axis xyz="-0.0 -1.0 0.000428"/>
-        <origin xyz="-0.09964 -0.06636 2.8e-05" rpy="0 0 0"/>
+        <origin xyz="-0.09964 -0.06636 0.0" rpy="0 0 0"/>
         <parent link="FL_hip_link"/>
         <child link="FL_uleg_link"/>
-        <xacro:uleg_limits></xacro:uleg_limits>
+        <axis xyz="-0.0 -1.0 -0.0"/>
+        <limit upper="0.785398" lower="-2.356194" effort="100" velocity="100"/>
         <xacro:if value="${use_dynamics}">
             <xacro:uleg_joint_dynamics></xacro:uleg_joint_dynamics>
@@ -85,9 +85,9 @@
     <!-- *********  BR_uleg  ********* -->
     <joint name="BR_uleg_joint" type="revolute">
-        <axis xyz="0.0 0.999996 0.002806"/>
-        <origin xyz="0.09964 0.066359 0.000186" rpy="0 0 0"/>
+        <origin xyz="0.09964 0.06636 0.0" rpy="0 0 0"/>
         <parent link="BR_hip_link"/>
         <child link="BR_uleg_link"/>
-        <xacro:uleg_limits></xacro:uleg_limits>
+        <axis xyz="-0.0 1.0 -0.0"/>
+        <limit upper="0.785398" lower="-2.356194" effort="100" velocity="100"/>
         <xacro:if value="${use_dynamics}">
             <xacro:uleg_joint_dynamics></xacro:uleg_joint_dynamics>
@@ -96,9 +96,9 @@
     <!-- *********  BL_uleg  ********* -->
     <joint name="BL_uleg_joint" type="revolute">
-        <axis xyz="0.0 1.0 -0.0"/>
         <origin xyz="0.09964 -0.06636 0.0" rpy="0 0 0"/>
         <parent link="BL_hip_link"/>
         <child link="BL_uleg_link"/>
-        <xacro:uleg_limits></xacro:uleg_limits>
+        <axis xyz="0.0 1.0 0.0"/>
+        <limit upper="0.785398" lower="-2.356194" effort="100" velocity="100"/>
         <xacro:if value="${use_dynamics}">
             <xacro:uleg_joint_dynamics></xacro:uleg_joint_dynamics>
@@ -107,9 +107,9 @@
     <!-- *********  FR_lleg  ********* -->
     <joint name="FR_lleg_joint" type="revolute">
-        <axis xyz="-0.0 -0.999043 -0.043739"/>
-        <origin xyz="0.143094 0.087993 -0.135091" rpy="0 0 0"/>
+        <origin xyz="0.140968 0.082 -0.140969" rpy="0 0 0"/>
         <parent link="FR_uleg_link"/>
         <child link="FR_lleg_link"/>
-        <xacro:lleg_limits></xacro:lleg_limits>
+        <axis xyz="-0.0 -1.0 0.0"/>
+        <limit upper="3.839724" lower="-0.698132" effort="100" velocity="100"/>
         <xacro:if value="${use_dynamics}">
             <xacro:lleg_joint_dynamics></xacro:lleg_joint_dynamics>
@@ -118,9 +118,9 @@
     <!-- *********  FL_lleg  ********* -->
     <joint name="FL_lleg_joint" type="revolute">
-        <axis xyz="-0.0 -1.0 0.000428"/>
-        <origin xyz="0.164113 -0.082048 -0.113151" rpy="0 0 0"/>
+        <origin xyz="0.140968 -0.082 -0.140968" rpy="0 0 0"/>
         <parent link="FL_uleg_link"/>
         <child link="FL_lleg_link"/>
-        <xacro:lleg_limits></xacro:lleg_limits>
+        <axis xyz="-0.0 -1.0 -0.0"/>
+        <limit upper="3.839724" lower="-0.698132" effort="100" velocity="100"/>
         <xacro:if value="${use_dynamics}">
             <xacro:lleg_joint_dynamics></xacro:lleg_joint_dynamics>
@@ -129,9 +129,9 @@
     <!-- *********  BR_lleg  ********* -->
     <joint name="BR_lleg_joint" type="revolute">
-        <origin xyz="-0.139215 0.0824 -0.14247" rpy="0 0 0"/>
+        <origin xyz="-0.140969 0.082 -0.140968" rpy="0 0 0"/>
         <parent link="BR_uleg_link"/>
         <child link="BR_lleg_link"/>
-        <axis xyz="0.0 0.999996 0.002806"/>
-        <xacro:lleg_limits></xacro:lleg_limits>
+        <axis xyz="-0.0 1.0 -0.0"/>
+        <limit upper="3.839724" lower="-0.698132" effort="100" velocity="100"/>
         <xacro:if value="${use_dynamics}">
             <xacro:lleg_joint_dynamics></xacro:lleg_joint_dynamics>
@@ -140,9 +140,9 @@
     <!-- *********  BL_lleg  ********* -->
     <joint name="BL_lleg_joint" type="revolute">
-        <axis xyz="0.0 1.0 -0.0"/>
-        <origin xyz="-0.140969 -0.082 -0.140969" rpy="0 0 0"/>
+        <origin xyz="-0.140969 -0.082 -0.140968" rpy="0 0 0"/>
         <parent link="BL_uleg_link"/>
         <child link="BL_lleg_link"/>
-        <xacro:lleg_limits></xacro:lleg_limits>
+        <axis xyz="0.0 1.0 0.0"/>
+        <limit upper="3.839724" lower="-0.698132" effort="100" velocity="100"/>
         <xacro:if value="${use_dynamics}">
             <xacro:lleg_joint_dynamics></xacro:lleg_joint_dynamics>
