Commit message: Updated the opendog_description: launch, urdf, meshes.

File: opendog_description/urdf/opendog_links.xacro (robot description, xacro)
@@ -28,5 +28,5 @@
     <link name="base_link">
         <inertial>
-          <origin xyz="0.2952464243198414 -0.07744895683312651 0.2642167275872589" rpy="0 0 0"/>
+          <origin xyz="0.2749797958231685 -0.08799492490648385 0.36444405374780864" rpy="0 0 0"/>
           <mass value="5"/>
           <inertia ixx="0.761631" iyy="4.077449" izz="3.905689" ixy="-0.001055" iyz="-0.000345" ixz="0.05479"/>
@@ -49,18 +49,18 @@
     <link name="FR_hip_link">
         <inertial>
-            <origin xyz="-0.0978580055625883 0.022211154148892714 0.0011350968600437605" rpy="0 0 0"/>
+            <origin xyz="-0.09804953144426388 0.01537887460379041 0.00019055475909179886" rpy="0 0 0"/>
             <mass value="2"/>
             <inertia ixx="0.012708" iyy="0.026996" izz="0.026264" ixy="-0.000651" iyz="8.1e-05" ixz="-1.7e-05"/>
         </inertial>
         <visual>
-            <origin xyz="-0.120789 0.018307 -0.263166" rpy="0 0 0"/>
-            <geometry>
-              <mesh filename="file://$(find opendog_description)/meshes/ur_shoulder_1.stl" scale="0.001 0.001 0.001"/>
-            </geometry>
-        </visual>
-        <collision>
-            <origin xyz="-0.120789 0.018307 -0.263166" rpy="0 0 0"/>
-            <geometry>
-              <mesh filename="file://$(find opendog_description)/meshes/ur_shoulder_1.stl" scale="0.001 0.001 0.001"/>
+            <origin xyz="-0.005372 0.029025 -0.34267" rpy="0 0 0"/>
+            <geometry>
+              <mesh filename="file://$(find opendog_description)/meshes/FR_hip_link_2.stl" scale="0.001 0.001 0.001"/>
+            </geometry>
+        </visual>
+        <collision>
+            <origin xyz="-0.005372 0.029025 -0.34267" rpy="0 0 0"/>
+            <geometry>
+              <mesh filename="file://$(find opendog_description)/meshes/FR_hip_link_2.stl" scale="0.001 0.001 0.001"/>
             </geometry>
         </collision>
@@ -69,18 +69,18 @@
     <link name="FL_hip_link">
         <inertial>
-            <origin xyz="-0.09797126193747194 -0.02210793721336457 0.00017264300535746457" rpy="0 0 0"/>
+            <origin xyz="-0.09804956975710932 -0.015379348802188275 0.00019128110374050378" rpy="0 0 0"/>
             <mass value="2"/>
             <inertia ixx="0.012737" iyy="0.027034" izz="0.026319" ixy="0.000689" iyz="-4.8e-05" ixz="1.1e-05"/>
         </inertial>
         <visual>
-            <origin xyz="-0.120789 0.136588 -0.263166" rpy="0 0 0"/>
-            <geometry>
-              <mesh filename="file://$(find opendog_description)/meshes/ul_shoulder_1.stl" scale="0.001 0.001 0.001"/>
-            </geometry>
-        </visual>
-        <collision>
-            <origin xyz="-0.120789 0.136588 -0.263166" rpy="0 0 0"/>
-            <geometry>
-              <mesh filename="file://$(find opendog_description)/meshes/ul_shoulder_1.stl" scale="0.001 0.001 0.001"/>
+            <origin xyz="-0.005091 0.147198 -0.340765" rpy="0 0 0"/>
+            <geometry>
+              <mesh filename="file://$(find opendog_description)/meshes/FL_hip_link_2.stl" scale="0.001 0.001 0.001"/>
+            </geometry>
+        </visual>
+        <collision>
+            <origin xyz="-0.005091 0.147198 -0.340765" rpy="0 0 0"/>
+            <geometry>
+              <mesh filename="file://$(find opendog_description)/meshes/FL_hip_link_2.stl" scale="0.001 0.001 0.001"/>
             </geometry>
         </collision>
@@ -89,18 +89,18 @@
     <link name="BR_hip_link">
         <inertial>
-            <origin xyz="0.09785770638545477 0.022239015222669276 0.0002249055293677138" rpy="0 0 0"/>
+            <origin xyz="0.09804922989186687 0.015379343283856973 0.00019128110374272422" rpy="0 0 0"/>
             <mass value="2"/>
             <inertia ixx="0.012708" iyy="0.027002" izz="0.026258" ixy="0.000651" iyz="5e-05" ixz="-1e-05"/>
         </inertial>
         <visual>
-            <origin xyz="-0.468789 0.018307 -0.263166" rpy="0 0 0"/>
-            <geometry>
-              <mesh filename="file://$(find opendog_description)/meshes/lr_hip_1.stl" scale="0.001 0.001 0.001"/>
-            </geometry>
-        </visual>
-        <collision>
-            <origin xyz="-0.468789 0.018307 -0.263166" rpy="0 0 0"/>
-            <geometry>
-              <mesh filename="file://$(find opendog_description)/meshes/lr_hip_1.stl" scale="0.001 0.001 0.001"/>
+            <origin xyz="-0.471531 0.028918 -0.340765" rpy="0 0 0"/>
+            <geometry>
+              <mesh filename="file://$(find opendog_description)/meshes/BR_hip_link_2.stl" scale="0.001 0.001 0.001"/>
+            </geometry>
+        </visual>
+        <collision>
+            <origin xyz="-0.471531 0.028918 -0.340765" rpy="0 0 0"/>
+            <geometry>
+              <mesh filename="file://$(find opendog_description)/meshes/BR_hip_link_2.stl" scale="0.001 0.001 0.001"/>
             </geometry>
         </collision>
@@ -109,18 +109,18 @@
     <link name="BL_hip_link">
         <inertial>
-            <origin xyz="0.09785589272231132 -0.02214347440508449 0.00015857382629103078" rpy="0 0 0"/>
+            <origin xyz="0.09804922228400342 -0.015379345578511366 0.00019128032686782648" rpy="0 0 0"/>
             <mass value="2"/>
             <inertia ixx="0.012784" iyy="0.027006" izz="0.026333" ixy="-0.000657" iyz="-4.9e-05" ixz="-1.1e-05"/>
         </inertial>
         <visual>
-            <origin xyz="-0.468789 0.136588 -0.263166" rpy="0 0 0"/>
-            <geometry>
-              <mesh filename="file://$(find opendog_description)/meshes/ll_hip_1.stl" scale="0.001 0.001 0.001"/>
-            </geometry>
-        </visual>
-        <collision>
-            <origin xyz="-0.468789 0.136588 -0.263166" rpy="0 0 0"/>
-            <geometry>
-              <mesh filename="file://$(find opendog_description)/meshes/ll_hip_1.stl" scale="0.001 0.001 0.001"/>
+            <origin xyz="-0.471531 0.147198 -0.340765" rpy="0 0 0"/>
+            <geometry>
+              <mesh filename="file://$(find opendog_description)/meshes/BL_hip_link_2.stl" scale="0.001 0.001 0.001"/>
+            </geometry>
+        </visual>
+        <collision>
+            <origin xyz="-0.471531 0.147198 -0.340765" rpy="0 0 0"/>
+            <geometry>
+              <mesh filename="file://$(find opendog_description)/meshes/BL_hip_link_2.stl" scale="0.001 0.001 0.001"/>
             </geometry>
         </collision>
@@ -130,18 +130,18 @@
     <link name="FR_uleg_link">
         <inertial>
-            <origin xyz="0.02695714675071178 0.0558355231259501 -0.02405284229057822" rpy="0 0 0"/>
+            <origin xyz="0.024785646151847765 0.06031237152858331 -0.02501775170684245" rpy="0 0 0"/>
             <mass value="2.7"/>
             <inertia ixx="0.060385" iyy="0.086191" izz="0.061956" ixy="0.004251" iyz="-0.003909" ixz="0.027901"/>
         </inertial>
         <visual>
-            <origin xyz="-0.021149 -0.047989 -0.266068" rpy="0 0 0"/>
-            <geometry>
-              <mesh filename="file://$(find opendog_description)/meshes/ur_middleleg_1.stl" scale="0.001 0.001 0.001"/>
-            </geometry>
-        </visual>
-        <collision>
-            <origin xyz="-0.021149 -0.047989 -0.266068" rpy="0 0 0"/>
-            <geometry>
-              <mesh filename="file://$(find opendog_description)/meshes/ur_middleleg_1.stl" scale="0.001 0.001 0.001"/>
+            <origin xyz="0.094268 -0.037335 -0.34267" rpy="0 0 0"/>
+            <geometry>
+              <mesh filename="file://$(find opendog_description)/meshes/FR_uleg_link_2.stl" scale="0.001 0.001 0.001"/>
+            </geometry>
+        </visual>
+        <collision>
+            <origin xyz="0.094268 -0.037335 -0.34267" rpy="0 0 0"/>
+            <geometry>
+              <mesh filename="file://$(find opendog_description)/meshes/FR_uleg_link_2.stl" scale="0.001 0.001 0.001"/>
             </geometry>
         </collision>
@@ -150,18 +150,18 @@
     <link name="FL_uleg_link">
         <inertial>
-            <origin xyz="0.03096990835496126 -0.05473890368922821 -0.021616826562582653" rpy="0 0 0"/>
+            <origin xyz="0.02578305194465416 -0.06037459079064242 -0.02602287407328735" rpy="0 0 0"/>
             <mass value="2.7"/>
             <inertia ixx="0.051391" iyy="0.085806" izz="0.071334" ixy="-0.006201" iyz="0.003973" ixz="0.025851"/>
         </inertial>
         <visual>
-            <origin xyz="-0.021149 0.202948 -0.263194" rpy="0 0 0"/>
-            <geometry>
-              <mesh filename="file://$(find opendog_description)/meshes/ul_middleleg_1.stl" scale="0.001 0.001 0.001"/>
-            </geometry>
-        </visual>
-        <collision>
-            <origin xyz="-0.021149 0.202948 -0.263194" rpy="0 0 0"/>
-            <geometry>
-              <mesh filename="file://$(find opendog_description)/meshes/ul_middleleg_1.stl" scale="0.001 0.001 0.001"/>
+            <origin xyz="0.094549 0.213558 -0.340765" rpy="0 0 0"/>
+            <geometry>
+              <mesh filename="file://$(find opendog_description)/meshes/FL_uleg_link_2.stl" scale="0.001 0.001 0.001"/>
+            </geometry>
+        </visual>
+        <collision>
+            <origin xyz="0.094549 0.213558 -0.340765" rpy="0 0 0"/>
+            <geometry>
+              <mesh filename="file://$(find opendog_description)/meshes/FL_uleg_link_2.stl" scale="0.001 0.001 0.001"/>
             </geometry>
         </collision>
@@ -170,18 +170,18 @@
     <link name="BR_uleg_link">
         <inertial>
-            <origin xyz="-0.0262175718604698 0.05480638461580738 -0.027051181506407118" rpy="0 0 0"/>
+            <origin xyz="-0.02478596816754486 0.060312838896795826 -0.025017037989093105" rpy="0 0 0"/>
             <mass value="2.7"/>
             <inertia ixx="0.061911" iyy="0.085831" izz="0.060788" ixy="-0.005251" iyz="-0.005031" ixz="-0.027715"/>
         </inertial>
         <visual>
-            <origin xyz="-0.568429 -0.048052 -0.263352" rpy="0 0 0"/>
-            <geometry>
-              <mesh filename="file://$(find opendog_description)/meshes/lr_middleleg_1.stl" scale="0.001 0.001 0.001"/>
-            </geometry>
-        </visual>
-        <collision>
-            <origin xyz="-0.568429 -0.048052 -0.263352" rpy="0 0 0"/>
-            <geometry>
-              <mesh filename="file://$(find opendog_description)/meshes/lr_middleleg_1.stl" scale="0.001 0.001 0.001"/>
+            <origin xyz="-0.571171 -0.037442 -0.340765" rpy="0 0 0"/>
+            <geometry>
+              <mesh filename="file://$(find opendog_description)/meshes/BR_uleg_link_2.stl" scale="0.001 0.001 0.001"/>
+            </geometry>
+        </visual>
+        <collision>
+            <origin xyz="-0.571171 -0.037442 -0.340765" rpy="0 0 0"/>
+            <geometry>
+              <mesh filename="file://$(find opendog_description)/meshes/BR_uleg_link_2.stl" scale="0.001 0.001 0.001"/>
             </geometry>
         </collision>
@@ -190,18 +190,18 @@
     <link name="BL_uleg_link">
         <inertial>
-            <origin xyz="-0.026552103840778662 -0.054729650997543317 -0.026879014160538728" rpy="0 0 0"/>
+            <origin xyz="-0.024912930584652382 -0.06035054910971113 -0.02514445341334004" rpy="0 0 0"/>
             <mass value="2.7"/>
             <inertia ixx="0.061226" iyy="0.085803" izz="0.061502" ixy="0.005391" iyz="0.005035" ixz="-0.027705"/>
         </inertial>
         <visual>
-            <origin xyz="-0.568429 0.202948 -0.263166" rpy="0 0 0"/>
-            <geometry>
-              <mesh filename="file://$(find opendog_description)/meshes/ll_middleleg_1.stl" scale="0.001 0.001 0.001"/>
-            </geometry>
-        </visual>
-        <collision>
-            <origin xyz="-0.568429 0.202948 -0.263166" rpy="0 0 0"/>
-            <geometry>
-              <mesh filename="file://$(find opendog_description)/meshes/ll_middleleg_1.stl" scale="0.001 0.001 0.001"/>
+            <origin xyz="-0.571171 0.213558 -0.340765" rpy="0 0 0"/>
+            <geometry>
+              <mesh filename="file://$(find opendog_description)/meshes/BL_uleg_link_2.stl" scale="0.001 0.001 0.001"/>
+            </geometry>
+        </visual>
+        <collision>
+            <origin xyz="-0.571171 0.213558 -0.340765" rpy="0 0 0"/>
+            <geometry>
+              <mesh filename="file://$(find opendog_description)/meshes/BL_uleg_link_2.stl" scale="0.001 0.001 0.001"/>
             </geometry>
         </collision>
@@ -211,18 +211,18 @@
     <link name="FR_lleg_link">
         <inertial>
-            <origin xyz="-0.05977620454383023 -0.03838893551235807 -0.041628896795266934" rpy="0 0 0"/>
+            <origin xyz="-0.06309907279078683 -0.04027150228827056 -0.06310352710956241" rpy="0 0 0"/>
             <mass value="0.3"/>
             <inertia ixx="0.007726" iyy="0.021253" izz="0.015039" ixy="0.000248" iyz="0.00018" ixz="-0.008798"/>
         </inertial>
         <visual>
-            <origin xyz="-0.164243 -0.135982 -0.130977" rpy="0 0 0"/>
-            <geometry>
-              <mesh filename="file://$(find opendog_description)/meshes/ur_lowerleg_1.stl" scale="0.001 0.001 0.001"/>
-            </geometry>
-        </visual>
-        <collision>
-            <origin xyz="-0.164243 -0.135982 -0.130977" rpy="0 0 0"/>
-            <geometry>
-              <mesh filename="file://$(find opendog_description)/meshes/ur_lowerleg_1.stl" scale="0.001 0.001 0.001"/>
+            <origin xyz="-0.0467 -0.119335 -0.201701" rpy="0 0 0"/>
+            <geometry>
+              <mesh filename="file://$(find opendog_description)/meshes/FR_lleg_link_2.stl" scale="0.001 0.001 0.001"/>
+            </geometry>
+        </visual>
+        <collision>
+            <origin xyz="-0.0467 -0.119335 -0.201701" rpy="0 0 0"/>
+            <geometry>
+              <mesh filename="file://$(find opendog_description)/meshes/FR_lleg_link_2.stl" scale="0.001 0.001 0.001"/>
             </geometry>
         </collision>
@@ -231,18 +231,18 @@
     <link name="FL_lleg_link">
         <inertial>
-            <origin xyz="-0.06724699359315146 0.04018076418942282 -0.048053981913996055" rpy="0 0 0"/>
+            <origin xyz="-0.06309910896868268 0.04027103185737707 -0.06310379848106407" rpy="0 0 0"/>
             <mass value="0.3"/>
             <inertia ixx="0.010996" iyy="0.029242" izz="0.019764" ixy="0.000158" iyz="0.000113" ixz="-0.012783"/>
         </inertial>
         <visual>
-            <origin xyz="-0.185262 0.284996 -0.150043" rpy="0 0 0"/>
-            <geometry>
-              <mesh filename="file://$(find opendog_description)/meshes/ul_lowerleg_1.stl" scale="0.001 0.001 0.001"/>
-            </geometry>
-        </visual>
-        <collision>
-            <origin xyz="-0.185262 0.284996 -0.150043" rpy="0 0 0"/>
-            <geometry>
-              <mesh filename="file://$(find opendog_description)/meshes/ul_lowerleg_1.stl" scale="0.001 0.001 0.001"/>
+            <origin xyz="-0.046419 0.295558 -0.199797" rpy="0 0 0"/>
+            <geometry>
+              <mesh filename="file://$(find opendog_description)/meshes/FL_lleg_link_2.stl" scale="0.001 0.001 0.001"/>
+            </geometry>
+        </visual>
+        <collision>
+            <origin xyz="-0.046419 0.295558 -0.199797" rpy="0 0 0"/>
+            <geometry>
+              <mesh filename="file://$(find opendog_description)/meshes/FL_lleg_link_2.stl" scale="0.001 0.001 0.001"/>
             </geometry>
         </collision>
@@ -251,18 +251,18 @@
     <link name="BR_lleg_link">
         <inertial>
-            <origin xyz="0.062326463733643256 -0.04007198062978043 -0.03590980750154857" rpy="0 0 0"/>
+            <origin xyz="0.06309976910343829 -0.04027103737571108 -0.06310379848106251" rpy="0 0 0"/>
             <mass value="0.3"/>
             <inertia ixx="0.006577" iyy="0.021257" izz="0.016183" ixy="0.00012" iyz="-6.8e-05" ixz="0.00823"/>
         </inertial>
         <visual>
-            <origin xyz="-0.429214 -0.130452 -0.120882" rpy="0 0 0"/>
-            <geometry>
-              <mesh filename="file://$(find opendog_description)/meshes/lr_lowerleg_2.stl" scale="0.001 0.001 0.001"/>
-            </geometry>
-        </visual>
-        <collision>
-            <origin xyz="-0.429214 -0.130452 -0.120882" rpy="0 0 0"/>
-            <geometry>
-              <mesh filename="file://$(find opendog_description)/meshes/lr_lowerleg_2.stl" scale="0.001 0.001 0.001"/>
+            <origin xyz="-0.430202 -0.119442 -0.199797" rpy="0 0 0"/>
+            <geometry>
+              <mesh filename="file://$(find opendog_description)/meshes/BR_lleg_link_2.stl" scale="0.001 0.001 0.001"/>
+            </geometry>
+        </visual>
+        <collision>
+            <origin xyz="-0.430202 -0.119442 -0.199797" rpy="0 0 0"/>
+            <geometry>
+              <mesh filename="file://$(find opendog_description)/meshes/BR_lleg_link_2.stl" scale="0.001 0.001 0.001"/>
             </geometry>
         </collision>
@@ -271,18 +271,18 @@
     <link name="BL_lleg_link">
         <inertial>
-            <origin xyz="0.06224424376041954 0.04017328339327439 -0.03594025105485621" rpy="0 0 0"/>
+            <origin xyz="0.06309976363052966 0.040271031313545036 -0.06310380154178746" rpy="0 0 0"/>
             <mass value="0.3"/>
             <inertia ixx="0.006615" iyy="0.021256" izz="0.016145" ixy="-0.000143" iyz="8.3e-05" ixz="0.008252"/>
         </inertial>
         <visual>
-            <origin xyz="-0.42746 0.284948 -0.122197" rpy="0 0 0"/>
-            <geometry>
-              <mesh filename="file://$(find opendog_description)/meshes/ll_lowerLeg_1.stl" scale="0.001 0.001 0.001"/>
-            </geometry>
-        </visual>
-        <collision>
-            <origin xyz="-0.42746 0.284948 -0.122197" rpy="0 0 0"/>
-            <geometry>
-              <mesh filename="file://$(find opendog_description)/meshes/ll_lowerLeg_1.stl" scale="0.001 0.001 0.001"/>
+            <origin xyz="-0.430202 0.295558 -0.199797" rpy="0 0 0"/>
+            <geometry>
+              <mesh filename="file://$(find opendog_description)/meshes/BL_lleg_link_2.stl" scale="0.001 0.001 0.001"/>
+            </geometry>
+        </visual>
+        <collision>
+            <origin xyz="-0.430202 0.295558 -0.199797" rpy="0 0 0"/>
+            <geometry>
+              <mesh filename="file://$(find opendog_description)/meshes/BL_lleg_link_2.stl" scale="0.001 0.001 0.001"/>
             </geometry>
             <surface>
