Commit message: Removed old macros

File: opendog_description/urdf/opendog_joints.xacro (robot description, xacro)
@@ -2,14 +2,4 @@
 <robot xmlns:xacro="http://www.ros.org/wiki/xacro">
     <xacro:include filename="consts.xacro" />
-    <!-- Limits -->
-    <xacro:macro name="hip_limits">
-        <limit lower="${hip_low_limit}" upper="${hip_up_limit}" velocity="${velocity}" effort="${effort}"/> <!-- effort = 7 -->
-    </xacro:macro>
-    <xacro:macro name="uleg_limits">
-        <limit lower="${uleg_low_limit}" upper="${uleg_up_limit}" velocity="${velocity}" effort="${effort}"/>
-    </xacro:macro>
-    <xacro:macro name="lleg_limits">
-        <limit lower="${lleg_low_limit}" upper="${lleg_up_limit}" velocity="${velocity}" effort="${effort}"/>
-    </xacro:macro>
     <!-- ******** world to base joint ********** -->
     <joint name="world_to_base" type="fixed">
@@ -23,8 +13,5 @@
         <child link="FR_hip_link"/>
         <axis xyz="1.0 -0.0 0.0"/>
-  <limit upper="0.174533" lower="-0.174533" effort="100" velocity="100"/>
-        <xacro:if value="${use_dynamics}">
-            <xacro:hip_joint_dynamics></xacro:hip_joint_dynamics>
-        </xacro:if>
+        <limit upper="0.174533" lower="-0.174533" effort="100" velocity="100"/>
     </joint>
     <!-- *********  FL_hip  ********* -->
@@ -35,7 +22,4 @@
         <axis xyz="-1.0 0.0 -0.0"/>
         <limit upper="0.174533" lower="-0.174533" effort="100" velocity="100"/>
-        <xacro:if value="${use_dynamics}">
-            <xacro:hip_joint_dynamics></xacro:hip_joint_dynamics>
-        </xacro:if>
     </joint>
     <!-- *********  BR_hip  ********* -->
@@ -46,7 +30,4 @@
         <axis xyz="1.0 -0.0 -0.0"/>
         <limit upper="0.174533" lower="-0.174533" effort="100" velocity="100"/>
-        <xacro:if value="${use_dynamics}">
-            <xacro:hip_joint_dynamics></xacro:hip_joint_dynamics>
-        </xacro:if>
     </joint>
     <!-- *********  BL_hip  ********* -->
@@ -57,7 +38,4 @@
         <axis xyz="-1.0 0.0 0.0"/>
         <limit upper="0.174533" lower="-0.174533" effort="100" velocity="100"/>
-        <xacro:if value="${use_dynamics}">
-            <xacro:hip_joint_dynamics></xacro:hip_joint_dynamics>
-        </xacro:if>
     </joint>
     <!-- *********  FR_uleg joint ********* -->
@@ -68,7 +46,4 @@
         <axis xyz="-0.0 -1.0 0.0"/>
         <limit upper="0.785398" lower="-2.356194" effort="100" velocity="100"/>
-        <xacro:if value="${use_dynamics}">
-            <xacro:uleg_joint_dynamics></xacro:uleg_joint_dynamics>
-        </xacro:if>
     </joint>
     <!-- *********  FL_uleg  ********* -->
@@ -79,7 +54,4 @@
         <axis xyz="-0.0 -1.0 -0.0"/>
         <limit upper="0.785398" lower="-2.356194" effort="100" velocity="100"/>
-        <xacro:if value="${use_dynamics}">
-            <xacro:uleg_joint_dynamics></xacro:uleg_joint_dynamics>
-        </xacro:if>
     </joint>
     <!-- *********  BR_uleg  ********* -->
@@ -90,7 +62,4 @@
         <axis xyz="-0.0 1.0 -0.0"/>
         <limit upper="0.785398" lower="-2.356194" effort="100" velocity="100"/>
-        <xacro:if value="${use_dynamics}">
-            <xacro:uleg_joint_dynamics></xacro:uleg_joint_dynamics>
-        </xacro:if>
     </joint>
     <!-- *********  BL_uleg  ********* -->
@@ -101,7 +70,4 @@
         <axis xyz="0.0 1.0 0.0"/>
         <limit upper="0.785398" lower="-2.356194" effort="100" velocity="100"/>
-        <xacro:if value="${use_dynamics}">
-            <xacro:uleg_joint_dynamics></xacro:uleg_joint_dynamics>
-        </xacro:if>
     </joint>
     <!-- *********  FR_lleg  ********* -->
@@ -112,7 +78,4 @@
         <axis xyz="-0.0 -1.0 0.0"/>
         <limit upper="3.839724" lower="-0.698132" effort="100" velocity="100"/>
-        <xacro:if value="${use_dynamics}">
-            <xacro:lleg_joint_dynamics></xacro:lleg_joint_dynamics>
-        </xacro:if>
     </joint>
     <!-- *********  FL_lleg  ********* -->
@@ -123,7 +86,4 @@
         <axis xyz="-0.0 -1.0 -0.0"/>
         <limit upper="3.839724" lower="-0.698132" effort="100" velocity="100"/>
-        <xacro:if value="${use_dynamics}">
-            <xacro:lleg_joint_dynamics></xacro:lleg_joint_dynamics>
-        </xacro:if>
     </joint>
     <!-- *********  BR_lleg  ********* -->
@@ -134,7 +94,4 @@
         <axis xyz="-0.0 1.0 -0.0"/>
         <limit upper="3.839724" lower="-0.698132" effort="100" velocity="100"/>
-        <xacro:if value="${use_dynamics}">
-            <xacro:lleg_joint_dynamics></xacro:lleg_joint_dynamics>
-        </xacro:if>
     </joint>
     <!-- *********  BL_lleg  ********* -->
@@ -145,7 +102,4 @@
         <axis xyz="0.0 1.0 0.0"/>
         <limit upper="3.839724" lower="-0.698132" effort="100" velocity="100"/>
-        <xacro:if value="${use_dynamics}">
-            <xacro:lleg_joint_dynamics></xacro:lleg_joint_dynamics>
-        </xacro:if>
     </joint>
 </robot>

Commit message: Further testings on real robot

File: opendog_description/urdf/opendog_joints.xacro (robot description, xacro)
@@ -20,5 +20,5 @@
         <parent link="base_link"/>
         <child link="FL_hip_link"/>
-        <axis xyz="-1.0 0.0 -0.0"/>
+        <axis xyz="1.0 0.0 0.0"/>   <!-- -1.0 0.0 -0.0 -->
         <limit upper="0.174533" lower="-0.174533" effort="100" velocity="100"/>
     </joint>
@@ -28,5 +28,5 @@
         <parent link="base_link"/>
         <child link="BR_hip_link"/>
-        <axis xyz="1.0 -0.0 -0.0"/>
+        <axis xyz="1.0 0.0 0.0"/>
         <limit upper="0.174533" lower="-0.174533" effort="100" velocity="100"/>
     </joint>
@@ -100,5 +100,5 @@
         <parent link="BL_uleg_link"/>
         <child link="BL_lleg_link"/>
-        <axis xyz="0.0 1.0 0.0"/>
+        <axis xyz="0.0 -1.0 0.0"/>
         <limit upper="3.839724" lower="-0.698132" effort="100" velocity="100"/>
     </joint>
