Commit message: feat: implémentation de la position stand et ajout de la téléopération

File: opendog_description/urdf/opendog.urdf.xacro (robot description, xacro)
@@ -1,10 +1,22 @@
 <?xml version="1.0" ?>
 <robot name="opendog_nostand" xmlns:xacro="http://www.ros.org/wiki/xacro">
-<!-- Configuration of Robot Links-->
-<xacro:include filename="$(find opendog_description)/urdf/opendog_links.xacro" />
-<!-- Configuration of Robot Joints-->
-<xacro:include filename="$(find opendog_description)/urdf/opendog_joints.xacro" />
-<!-- Other Configurations-->
-<xacro:include filename="$(find opendog_description)/urdf/materials.xacro" />
-<xacro:include filename="$(find opendog_description)/urdf/opendog.trans" />
+  <!-- Argument optionnel pour activer l'injection des plugins Gazebo -->
+  <xacro:arg name="use_gazebo" default="false"/>
+  <!-- Configuration of Robot Links-->
+  <xacro:include filename="$(find opendog_description)/urdf/opendog_stand_links.xacro"/>
+  <xacro:include filename="$(find opendog_description)/urdf/opendog_stand_joints.xacro"/>
+  <!-- Configuration of Robot Joints -->
+  <xacro:include filename="$(find opendog_description)/urdf/opendog_links.xacro"/>
+  <xacro:include filename="$(find opendog_description)/urdf/opendog_joints.xacro"/>
+  <!-- Other Configurations -->
+  <xacro:include filename="$(find opendog_description)/urdf/materials.xacro"/>
+  <xacro:include filename="$(find opendog_description)/urdf/opendog.trans"/>
+  <!-- ros2_control configuration -->
+  <xacro:include filename="$(find opendog_description)/urdf/opendog_ros2_control.xacro"/>
+  <xacro:opendog_ros2_control name="opendog_hw"/>
+  <!-- Inclusion et appel conditionnels du plugin Gazebo -->
+  <xacro:if value="$(arg use_gazebo)">
+    <xacro:include filename="$(find opendog_description)/urdf/opendog_gazebo_control.xacro"/>
+    <xacro:opendog_gazebo_control name="opendog_hw_gazebo"/>
+  </xacro:if>
 </robot>

File: opendog_description/urdf/opendog_joints.xacro (robot description, xacro)
@@ -2,9 +2,4 @@
 <robot xmlns:xacro="http://www.ros.org/wiki/xacro">
     <xacro:include filename="consts.xacro" />
-    <!-- ******** world to base joint ********** -->
-    <joint name="world_to_base" type="fixed">
-        <parent link="base_link"/>
-        <child link="world"/>
-    </joint>
     <!-- *********  FR_hip joint ********* -->
     <joint name="FR_hip_joint" type="revolute">

File: opendog_description/urdf/opendog_links.xacro (robot description, xacro)
@@ -22,11 +22,8 @@
         <mesh filename="file://$(find opendog_description)/meshes/LLEG.stl" scale="0.001 0.001 0.001"/>
     </xacro:macro>
-    <!-- *********** Inertial link *********** -->
-    <link name="world">
-    </link>
     <!-- *********** base link *********** -->
     <link name="base_link">
         <inertial>
-          <origin xyz="0.2749797958231685 -0.08799492490648385 0.36444405374780864" rpy="0 0 0"/>
+          <origin xyz="0 0.0 0" rpy="0 0 0"/>
           <mass value="5"/>
           <inertia ixx="0.761631" iyy="4.077449" izz="3.905689" ixy="-0.001055" iyz="-0.000345" ixz="0.05479"/>

File: opendog_description/urdf/opendog_stand_joints.xacro (robot description, xacro)
@@ -1,90 +1,16 @@
 <?xml version="1.0" ?>
-<robot name="opendog_stand" xmlns:xacro="http://www.ros.org/wiki/xacro">
-<!-- Joints -->
-<joint name="fixed_to_world_joint" type="fixed">
-  <origin xyz="0 0 0" rpy="0 0 0"/>
+<robot xmlns:xacro="http://www.ros.org/wiki/xacro">
+    <!-- Joint entre world et stand -->
+<joint name="world_to_stand_link" type="fixed">
   <parent link="world"/>
+  <child link="stand_link"/>
+  <origin xyz="0 0 0.1" rpy="0 0 0"/> <!-- Centre du cylindre à 0.5m -->
+</joint>
+  <!-- Joint fixe entre stand et base_link -->
+<joint name="stand_to_base" type="fixed">
+  <origin xyz="0 0 0.3" rpy="0 0 0"/>
+  <!-- Positionné au sommet du stand (z=0.5 + 0.5 = 1m) -->
+  <parent link="stand_link"/>
   <child link="base_link"/>
 </joint>
-<joint name="ur_shoulder_to_base_link" type="revolute">
-  <origin xyz="-0.54228 0.109568 0.089167" rpy="0 0 0"/>
-  <parent link="base_linkr_1"/>
-  <child link="ur_shoulder_1"/>
-  <axis xyz="1.0 -0.0 0.0"/>
-  <limit upper="0.349066" lower="-0.349066" effort="100" velocity="100"/>
-</joint>
-<joint name="ur_upperleg_to_shoulder" type="continuous">
-  <origin xyz="-0.099641 0.06636 0.0" rpy="0 0 0"/>
-  <parent link="ur_shoulder_1"/>
-  <child link="ur_middleleg_1"/>
-  <axis xyz="-0.0 -1.0 -0.0"/>
-</joint>
-<joint name="ul_shoulder_to_base_link" type="revolute">
-  <origin xyz="-0.54228 -0.008713 0.089167" rpy="0 0 0"/>
-  <parent link="base_linkr_1"/>
-  <child link="ul_shoulder_1"/>
-  <axis xyz="-1.0 0.0 -0.0"/>
-  <limit upper="0.349066" lower="-0.785398" effort="100" velocity="100"/>
-</joint>
-<joint name="ul_upperleg_to_shoulder" type="continuous">
-  <origin xyz="-0.099641 -0.066359 0.0" rpy="0 0 0"/>
-  <parent link="ul_shoulder_1"/>
-  <child link="ul_middleleg_1"/>
-  <axis xyz="-0.0 -1.0 0.0"/>
-</joint>
-<joint name="ll_hip_to_base_link" type="revolute">
-  <origin xyz="-0.19428 -0.008713 0.089167" rpy="0 0 0"/>
-  <parent link="base_linkr_1"/>
-  <child link="ll_hip_1"/>
-  <axis xyz="-1.0 0.0 0.0"/>
-  <limit upper="0.436332" lower="-0.785398" effort="100" velocity="100"/>
-</joint>
-<joint name="ll_upperleg_to_hip" type="continuous">
-  <origin xyz="0.09964 -0.066359 0.0" rpy="0 0 0"/>
-  <parent link="ll_hip_1"/>
-  <child link="ll_middleleg_1"/>
-  <axis xyz="0.0 1.0 -0.0"/>
-</joint>
-<joint name="lr_hip_to_base_link" type="revolute">
-  <origin xyz="-0.19428 0.109568 0.089167" rpy="0 0 0"/>
-  <parent link="base_linkr_1"/>
-  <child link="lr_hip_1"/>
-  <axis xyz="1.0 -0.0 -0.0"/>
-  <limit upper="0.349066" lower="-0.785398" effort="100" velocity="100"/>
-</joint>
-<joint name="lr_upperleg_to_hip" type="continuous">
-  <origin xyz="0.09964 0.06636 0.0" rpy="0 0 0"/>
-  <parent link="lr_hip_1"/>
-  <child link="lr_middleleg_1"/>
-  <axis xyz="-0.0 1.0 0.0"/>
-</joint>
-<joint name="lr_lowerleg_to_upperleg" type="continuous">
-  <origin xyz="-0.128146 0.082 -0.152718" rpy="0 0 0"/>
-  <parent link="lr_middleleg_1"/>
-  <child link="lr_lowerleg_2"/>
-  <axis xyz="-0.0 1.0 0.0"/>
-</joint>
-<joint name="ll_lowerleg_to_upperleg" type="continuous">
-  <origin xyz="-0.140969 -0.082 -0.140968" rpy="0 0 0"/>
-  <parent link="ll_middleleg_1"/>
-  <child link="ll_lowerLeg_1"/>
-  <axis xyz="0.0 1.0 -0.0"/>
-</joint>
-<joint name="ul_lowerleg_to_upperleg" type="continuous">
-  <origin xyz="0.140969 -0.082 -0.140968" rpy="0 0 0"/>
-  <parent link="ul_middleleg_1"/>
-  <child link="ul_lowerleg_1"/>
-  <axis xyz="-0.0 -1.0 0.0"/>
-</joint>
-<joint name="ur_lowerleg_to_upperleg" type="continuous">
-  <origin xyz="0.140969 0.082 -0.140968" rpy="0 0 0"/>
-  <parent link="ur_middleleg_1"/>
-  <child link="ur_lowerleg_1"/>
-  <axis xyz="-0.0 -1.0 -0.0"/>
-</joint>
-<joint name="Rigid 28" type="fixed">
-  <origin xyz="0.665939 -0.117254 0.385318" rpy="0 0 0"/>
-  <parent link="base_link"/>
-  <child link="base_linkr_1"/>
-</joint>
 </robot>

File: opendog_description/urdf/opendog_stand_links.xacro (robot description, xacro)
@@ -1,271 +1,31 @@
 <?xml version="1.0" ?>
-<robot name="openleg" xmlns:xacro="http://www.ros.org/wiki/xacro">
-<!-- Robot Links -->
-<link name="world"/>
-<link name="base_link">
+<robot  xmlns:xacro="http://www.ros.org/wiki/xacro">
+ <!-- Définition du lien du stand -->
+ <!-- World link -->
+ <link name="world"/>
+ <!-- Stand link -->
+  <link name="stand_link">
   <visual>
-    <origin xyz="0 0 0" rpy="0 0 0"/>
-    <material name="silver"/>
-  </visual>
-</link>
-<link name="ur_shoulder_1">
-  <inertial>
-    <origin xyz="-0.09785829303628078 0.02223966584464055 0.00016305377611242067" rpy="0 0 0"/>
-    <mass value="8.21838423136781"/>
-    <inertia ixx="0.012708" iyy="0.027002" izz="0.026258" ixy="-0.000651" iyz="4.8e-05" ixz="1.1e-05"/>
-  </inertial>
-  <visual>
-    <origin xyz="-0.123659 0.007686 -0.474485" rpy="0 0 0"/>
     <geometry>
-      <mesh filename="file://$(find opendog_description)/meshes/ur_shoulder_1.stl" scale="0.001 0.001 0.001"/>
+      <box size="0.5 0.5 0.2"/>
     </geometry>
-    <material name="silver"/>
+    <material name="green"> <!-- Changez le nom pour éviter les conflits -->
+      <color rgba="0 0 0.8 1.0"/>
+    </material>
   </visual>
   <collision>
-    <origin xyz="-0.123659 0.007686 -0.474485" rpy="0 0 0"/>
     <geometry>
-      <mesh filename="file://$(find opendog_description)/meshes/ur_shoulder_1.stl" scale="0.001 0.001 0.001"/>
+      <box size="0.5 0.5 0.2"/>
     </geometry>
   </collision>
-</link>
-<link name="ur_middleleg_1">
   <inertial>
-    <origin xyz="0.02655252289271656 0.05472965720806993 -0.026878473024749328" rpy="0 0 0"/>
-    <mass value="14.227687011972318"/>
-    <inertia ixx="0.061226" iyy="0.085803" izz="0.061502" ixy="0.005391" iyz="-0.005035" ixz="0.027705"/>
+    <mass value="100"/>
+    <origin xyz="0 0 0"/>
+    <inertia ixx="1" iyy="1" izz="1" ixy="0" ixz="0" iyz="0"/>
   </inertial>
-  <visual>
-    <origin xyz="-0.024018 -0.058674 -0.474485" rpy="0 0 0"/>
-    <geometry>
-      <mesh filename="file://$(find opendog_description)/meshes/ur_middleleg_1.stl" scale="0.001 0.001 0.001"/>
-    </geometry>
-    <material name="silver"/>
-  </visual>
-  <collision>
-    <origin xyz="-0.024018 -0.058674 -0.474485" rpy="0 0 0"/>
-    <geometry>
-      <mesh filename="file://$(find opendog_description)/meshes/ur_middleleg_1.stl" scale="0.001 0.001 0.001"/>
-    </geometry>
-  </collision>
-</link>
-<link name="ul_shoulder_1">
-  <inertial>
-    <origin xyz="-0.09797154941116658 -0.022107897325156334 0.0001637293869130585" rpy="0 0 0"/>
-    <mass value="8.250541403982718"/>
-    <inertia ixx="0.012737" iyy="0.027034" izz="0.026319" ixy="0.000689" iyz="-4.7e-05" ixz="1.2e-05"/>
-  </inertial>
-  <visual>
-    <origin xyz="-0.123659 0.125967 -0.474485" rpy="0 0 0"/>
-    <geometry>
-      <mesh filename="file://$(find opendog_description)/meshes/ul_shoulder_1.stl" scale="0.001 0.001 0.001"/>
-    </geometry>
-    <material name="silver"/>
-  </visual>
-  <collision>
-    <origin xyz="-0.123659 0.125967 -0.474485" rpy="0 0 0"/>
-    <geometry>
-      <mesh filename="file://$(find opendog_description)/meshes/ul_shoulder_1.stl" scale="0.001 0.001 0.001"/>
-    </geometry>
-  </collision>
-</link>
-<link name="ul_middleleg_1">
-  <inertial>
-    <origin xyz="0.026552263666205788 -0.05473054768390884 -0.026878297131730566" rpy="0 0 0"/>
-    <mass value="14.227664566368246"/>
-    <inertia ixx="0.061226" iyy="0.085803" izz="0.061502" ixy="-0.005391" iyz="0.005035" ixz="0.027705"/>
-  </inertial>
-  <visual>
-    <origin xyz="-0.024018 0.192326 -0.474485" rpy="0 0 0"/>
-    <geometry>
-      <mesh filename="file://$(find opendog_description)/meshes/ul_middleleg_1.stl" scale="0.001 0.001 0.001"/>
-    </geometry>
-    <material name="silver"/>
-  </visual>
-  <collision>
-    <origin xyz="-0.024018 0.192326 -0.474485" rpy="0 0 0"/>
-    <geometry>
-      <mesh filename="file://$(find opendog_description)/meshes/ul_middleleg_1.stl" scale="0.001 0.001 0.001"/>
-    </geometry>
-  </collision>
-</link>
-<link name="ll_hip_1">
-  <inertial>
-    <origin xyz="0.0978556052486162 -0.022143362618367995 0.00015911556218167755" rpy="0 0 0"/>
-    <mass value="8.221636898406961"/>
-    <inertia ixx="0.012784" iyy="0.027006" izz="0.026333" ixy="-0.000657" iyz="-4.9e-05" ixz="-1.1e-05"/>
-  </inertial>
-  <visual>
-    <origin xyz="-0.471659 0.125967 -0.474485" rpy="0 0 0"/>
-    <geometry>
-      <mesh filename="file://$(find opendog_description)/meshes/ll_hip_1.stl" scale="0.001 0.001 0.001"/>
-    </geometry>
-    <material name="silver"/>
-  </visual>
-  <collision>
-    <origin xyz="-0.471659 0.125967 -0.474485" rpy="0 0 0"/>
-    <geometry>
-      <mesh filename="file://$(find opendog_description)/meshes/ll_hip_1.stl" scale="0.001 0.001 0.001"/>
-    </geometry>
-  </collision>
-</link>
-<link name="ll_middleleg_1">
-  <inertial>
-    <origin xyz="-0.02655239130407583 -0.05473053921082616 -0.026878472414248566" rpy="0 0 0"/>
-    <mass value="14.227687254589894"/>
-    <inertia ixx="0.061226" iyy="0.085803" izz="0.061502" ixy="0.005391" iyz="0.005035" ixz="-0.027705"/>
-  </inertial>
-  <visual>
-    <origin xyz="-0.571299 0.192326 -0.474485" rpy="0 0 0"/>
-    <geometry>
-      <mesh filename="file://$(find opendog_description)/meshes/ll_middleleg_1.stl" scale="0.001 0.001 0.001"/>
-    </geometry>
-    <material name="silver"/>
-  </visual>
-  <collision>
-    <origin xyz="-0.571299 0.192326 -0.474485" rpy="0 0 0"/>
-    <geometry>
-      <mesh filename="file://$(find opendog_description)/meshes/ll_middleleg_1.stl" scale="0.001 0.001 0.001"/>
-    </geometry>
-  </collision>
-</link>
-<link name="lr_hip_1">
-  <inertial>
-    <origin xyz="0.09785741891175764 0.022239671062088552 0.00016304661283195188" rpy="0 0 0"/>
-    <mass value="8.218386359006598"/>
-    <inertia ixx="0.012708" iyy="0.027002" izz="0.026258" ixy="0.000651" iyz="4.8e-05" ixz="-1.1e-05"/>
-  </inertial>
-  <visual>
-    <origin xyz="-0.471659 0.007686 -0.474485" rpy="0 0 0"/>
-    <geometry>
-      <mesh filename="file://$(find opendog_description)/meshes/lr_hip_1.stl" scale="0.001 0.001 0.001"/>
-    </geometry>
-    <material name="silver"/>
-  </visual>
-  <collision>
-    <origin xyz="-0.471659 0.007686 -0.474485" rpy="0 0 0"/>
-    <geometry>
-      <mesh filename="file://$(find opendog_description)/meshes/lr_hip_1.stl" scale="0.001 0.001 0.001"/>
-    </geometry>
-  </collision>
-</link>
-<link name="lr_middleleg_1">
-  <inertial>
-    <origin xyz="-0.02410854634893167 0.05472964093419624 -0.029090152760393895" rpy="0 0 0"/>
-    <mass value="14.2276519621801"/>
-    <inertia ixx="0.066039" iyy="0.085803" izz="0.056689" ixy="-0.004932" iyz="-0.005486" ixz="-0.027308"/>
-  </inertial>
-  <visual>
-    <origin xyz="-0.571299 -0.058674 -0.474485" rpy="0 0 0"/>
-    <geometry>
-      <mesh filename="file://$(find opendog_description)/meshes/lr_middleleg_1.stl" scale="0.001 0.001 0.001"/>
-    </geometry>
-    <material name="silver"/>
-  </visual>
-  <collision>
-    <origin xyz="-0.571299 -0.058674 -0.474485" rpy="0 0 0"/>
-    <geometry>
-      <mesh filename="file://$(find opendog_description)/meshes/lr_middleleg_1.stl" scale="0.001 0.001 0.001"/>
-    </geometry>
-  </collision>
-</link>
-<link name="lr_lowerleg_2">
-  <inertial>
-    <origin xyz="0.06224361192579653 -0.0401732772739245 -0.03594052661627556" rpy="0 0 0"/>
-    <mass value="4.0749496298790815"/>
-    <inertia ixx="0.006615" iyy="0.021256" izz="0.016145" ixy="0.000143" iyz="-8.3e-05" ixz="0.008252"/>
-  </inertial>
-  <visual>
-    <origin xyz="-0.443153 -0.140674 -0.321767" rpy="0 0 0"/>
-    <geometry>
-      <mesh filename="file://$(find opendog_description)/meshes/lr_lowerleg_2.stl" scale="0.001 0.001 0.001"/>
-    </geometry>
-    <material name="silver"/>
-  </visual>
-  <collision>
-    <origin xyz="-0.443153 -0.140674 -0.321767" rpy="0 0 0"/>
-    <geometry>
-      <mesh filename="file://$(find opendog_description)/meshes/lr_lowerleg_2.stl" scale="0.001 0.001 0.001"/>
-    </geometry>
-  </collision>
-</link>
-<link name="ll_lowerLeg_1">
-  <inertial>
-    <origin xyz="0.06224395628672491 0.04017239517999152 -0.0359407275155198" rpy="0 0 0"/>
-    <mass value="4.074949631235474"/>
-    <inertia ixx="0.006615" iyy="0.021256" izz="0.016145" ixy="-0.000143" iyz="8.3e-05" ixz="0.008252"/>
-  </inertial>
-  <visual>
-    <origin xyz="-0.43033 0.274326 -0.333517" rpy="0 0 0"/>
-    <geometry>
-      <mesh filename="file://$(find opendog_description)/meshes/ll_lowerLeg_1.stl" scale="0.001 0.001 0.001"/>
-    </geometry>
-    <material name="silver"/>
-  </visual>
-  <collision>
-    <origin xyz="-0.43033 0.274326 -0.333517" rpy="0 0 0"/>
-    <geometry>
-      <mesh filename="file://$(find opendog_description)/meshes/ll_lowerLeg_1.stl" scale="0.001 0.001 0.001"/>
-    </geometry>
-  </collision>
-</link>
-<link name="ul_lowerleg_1">
-  <inertial>
-    <origin xyz="-0.07156807198737279 0.04020081884647034 -0.041323948195093385" rpy="0 0 0"/>
-    <mass value="4.21995926358348"/>
-    <inertia ixx="0.008622" iyy="0.029242" izz="0.022138" ixy="0.000174" iyz="0.000101" ixz="-0.011703"/>
-  </inertial>
-  <visual>
-    <origin xyz="-0.164987 0.274326 -0.333517" rpy="0 0 0"/>
-    <geometry>
-      <mesh filename="file://$(find opendog_description)/meshes/ul_lowerleg_1.stl" scale="0.001 0.001 0.001"/>
-    </geometry>
-    <material name="silver"/>
-  </visual>
-  <collision>
-    <origin xyz="-0.164987 0.274326 -0.333517" rpy="0 0 0"/>
-    <geometry>
-      <mesh filename="file://$(find opendog_description)/meshes/ul_lowerleg_1.stl" scale="0.001 0.001 0.001"/>
-    </geometry>
-  </collision>
-</link>
-<link name="ur_lowerleg_1">
-  <inertial>
-    <origin xyz="-0.050820875236943314 -0.04017327621481369 -0.05082597628130897" rpy="0 0 0"/>
-    <mass value="4.07494961611928"/>
-    <inertia ixx="0.011379" iyy="0.021256" izz="0.011381" ixy="-0.000117" iyz="-0.000117" ixz="-0.009529"/>
-  </inertial>
-  <visual>
-    <origin xyz="-0.164987 -0.140674 -0.333517" rpy="0 0 0"/>
-    <geometry>
-      <mesh filename="file://$(find opendog_description)/meshes/ur_lowerleg_1.stl" scale="0.001 0.001 0.001"/>
-    </geometry>
-    <material name="silver"/>
-  </visual>
-  <collision>
-    <origin xyz="-0.164987 -0.140674 -0.333517" rpy="0 0 0"/>
-    <geometry>
-      <mesh filename="file://$(find opendog_description)/meshes/ur_lowerleg_1.stl" scale="0.001 0.001 0.001"/>
-    </geometry>
-  </collision>
-</link>
-<link name="base_linkr_1">
-  <inertial>
-    <origin xyz="-0.3678228631538539 0.05042615495359001 0.09021826931094556" rpy="0 0 0"/>
-    <mass value="70.88293840121786"/>
-    <inertia ixx="0.761631" iyy="4.077449" izz="3.905689" ixy="-0.001055" iyz="-0.000345" ixz="0.05479"/>
-  </inertial>
-  <visual>
-    <origin xyz="-0.665939 0.117254 -0.385318" rpy="0 0 0"/>
-    <geometry>
-      <mesh filename="file://$(find opendog_description)/meshes/base_linkr_1.stl" scale="0.001 0.001 0.001"/>
-    </geometry>
-    <material name="silver"/>
-  </visual>
-  <collision>
-    <origin xyz="-0.665939 0.117254 -0.385318" rpy="0 0 0"/>
-    <geometry>
-      <mesh filename="file://$(find opendog_description)/meshes/base_linkr_1.stl" scale="0.001 0.001 0.001"/>
-    </geometry>
-  </collision>
-</link>
+  </link>
+    <!-- Gazebo: rendre le stand statique pour éviter que le robot "tourne" dans la simulation -->
+    <gazebo reference="stand_link">
+      <static>true</static>
+    </gazebo>
 </robot>
