Commit message: WIP: BR/BL leg tests, gear_ratio + uleg axis fixes, pre-hyperdog-start-gates

File: opendog_description/urdf/opendog.urdf.xacro (robot description, xacro)
@@ -11,7 +11,7 @@
   <!-- ========================================= -->
   <!-- Configuration of Robot Links-->
-  <xacro:include filename="$(find opendog_description)/urdf/opendog_stand_links.xacro"/>
+  <!-- Configuration of Robot Joints -->
+    <xacro:include filename="$(find opendog_description)/urdf/opendog_stand_links.xacro"/>
   <xacro:include filename="$(find opendog_description)/urdf/opendog_stand_joints.xacro"/>
-  <!-- Configuration of Robot Joints -->
   <xacro:include filename="$(find opendog_description)/urdf/opendog_links.xacro"/>
   <xacro:include filename="$(find opendog_description)/urdf/opendog_joints.xacro"/>
@@ -22,4 +22,6 @@
   <!--     HARDWARE INTERFACE (CONDITIONNEL)    -->
   <!-- ========================================= -->
+  <!-- En mode gazebo, ne jamais charger l'interface hardware reelle (USB/CAN) -->
+<xacro:unless value="$(arg use_gazebo)">
   <!-- Choix entre USB et CAN -->
   <xacro:if value="$(arg use_can)">
@@ -33,10 +35,5 @@
     <xacro:opendog_ros2_control name="opendog_hw"/>
   </xacro:unless>
+</xacro:unless>
   <!-- ========================================= -->
-  <!--     SIMULATION GAZEBO (OPTIONNEL)        -->
-  <!-- ========================================= -->
-  <xacro:if value="$(arg use_gazebo)">
-    <xacro:include filename="$(find opendog_description)/urdf/opendog_gazebo.xacro"/>
-    <xacro:opendog_gazebo_control name="opendog_hw_gazebo"/>
-  </xacro:if>
 </robot>

File: opendog_description/urdf/opendog_joints.xacro (robot description, xacro)
@@ -39,6 +39,6 @@
         <parent link="FR_hip_link"/>
         <child link="FR_uleg_link"/>
-        <axis xyz="-0.0 -1.0 0.0"/>
-        <limit upper="0.785398" lower="-2.356194" effort="100" velocity="100"/>
+        <axis xyz="-0.0 1.0 0.0"/>
+        <limit upper="1.221730" lower="-2.356194" effort="100" velocity="100"/>
     </joint>
     <!-- *********  FL_uleg  ********* -->
@@ -47,6 +47,6 @@
         <parent link="FL_hip_link"/>
         <child link="FL_uleg_link"/>
-        <axis xyz="-0.0 -1.0 -0.0"/>
-        <limit upper="0.785398" lower="-2.356194" effort="100" velocity="100"/>
+        <axis xyz="-0.0 1.0 -0.0"/>
+        <limit upper="1.221730" lower="-2.356194" effort="100" velocity="100"/>
     </joint>
     <!-- *********  BR_uleg  ********* -->
@@ -55,6 +55,6 @@
         <parent link="BR_hip_link"/>
         <child link="BR_uleg_link"/>
-        <axis xyz="-0.0 1.0 -0.0"/>
-        <limit upper="0.785398" lower="-2.356194" effort="100" velocity="100"/>
+        <axis xyz="-0.0 -1.0 -0.0"/>
+        <limit upper="1.221730" lower="-2.356194" effort="100" velocity="100"/>
     </joint>
     <!-- *********  BL_uleg  ********* -->
@@ -63,6 +63,6 @@
         <parent link="BL_hip_link"/>
         <child link="BL_uleg_link"/>
-        <axis xyz="0.0 1.0 0.0"/>
-        <limit upper="0.785398" lower="-2.356194" effort="100" velocity="100"/>
+        <axis xyz="0.0 -1.0 0.0"/>
+        <limit upper="1.221730" lower="-2.356194" effort="100" velocity="100"/>
     </joint>
     <!-- *********  FR_lleg  ********* -->

File: opendog_description/urdf/opendog_stand_links.xacro (robot description, xacro)
@@ -25,5 +25,5 @@
   </inertial>
   </link>
-    <!-- Gazebo: rendre le stand statique pour éviter que le robot "tourne" dans la simulation -->
+    <!-- Gazebo - rendre le stand statique pour éviter que le robot "tourne" dans la simulation -->
     <gazebo reference="stand_link">
       <static>true</static>

File: opendog_gazebosim/description/gazebo_ros2_control_plugin.xacro (robot description, xacro)
@@ -10,4 +10,7 @@
                 <param name="min">-1.57</param>
                 <param name="max">1.57</param>
+                <param name="p">100.0</param>
+                <param name="i">0.0</param>
+                <param name="d">5.0</param>
             </command_interface>
             <state_interface name="position">
@@ -21,7 +24,10 @@
                 <param name="min">-1.2217</param>
                 <param name="max">3.14</param>
+                <param name="p">150.0</param>
+                <param name="i">0.0</param>
+                <param name="d">10.0</param>
             </command_interface>
             <state_interface name="position">
-                <param name="initial_value">0.0</param>
+                <param name="initial_value">-0.7854</param>
             </state_interface>
             <state_interface name="velocity"/>
@@ -32,7 +38,10 @@
                 <param name="min">0.45</param>
                 <param name="max">2.3562</param>
+                <param name="p">50.0</param>
+                <param name="i">0.0</param>
+                <param name="d">2.0</param>
             </command_interface>
             <state_interface name="position">
-                <param name="initial_value">0.45</param>
+                <param name="initial_value">0.0</param>
             </state_interface>
             <state_interface name="velocity"/>
@@ -43,4 +52,7 @@
                 <param name="min">-1.57</param>
                 <param name="max">1.57</param>
+                <param name="p">100.0</param>
+                <param name="i">0.0</param>
+                <param name="d">5.0</param>
             </command_interface>
             <state_interface name="position">
@@ -54,7 +66,10 @@
                 <param name="min">-1.2217</param>
                 <param name="max">3.14</param>
+                <param name="p">150.0</param>
+                <param name="i">0.0</param>
+                <param name="d">10.0</param>
             </command_interface>
             <state_interface name="position">
-                <param name="initial_value">0.0</param>
+                <param name="initial_value">-0.7854</param>
             </state_interface>
             <state_interface name="velocity"/>
@@ -65,7 +80,10 @@
                 <param name="min">0.45</param>
                 <param name="max">2.3562</param>
+                <param name="p">50.0</param>
+                <param name="i">0.0</param>
+                <param name="d">2.0</param>
             </command_interface>
             <state_interface name="position">
-                <param name="initial_value">0.45</param>
+                <param name="initial_value">0.0</param>
             </state_interface>
             <state_interface name="velocity"/>
@@ -76,4 +94,7 @@
                 <param name="min">-1.57</param>
                 <param name="max">1.57</param>
+                <param name="p">100.0</param>
+                <param name="i">0.0</param>
+                <param name="d">5.0</param>
             </command_interface>
             <state_interface name="position">
@@ -87,7 +108,10 @@
                 <param name="min">-1.2217</param>
                 <param name="max">3.14</param>
+                <param name="p">150.0</param>
+                <param name="i">0.0</param>
+                <param name="d">10.0</param>
             </command_interface>
             <state_interface name="position">
-                <param name="initial_value">0.0</param>
+                <param name="initial_value">-0.7854</param>
             </state_interface>
             <state_interface name="velocity"/>
@@ -98,7 +122,10 @@
                 <param name="min">0.45</param>
                 <param name="max">2.3562</param>
+                <param name="p">50.0</param>
+                <param name="i">0.0</param>
+                <param name="d">2.0</param>
             </command_interface>
             <state_interface name="position">
-                <param name="initial_value">0.45</param>
+                <param name="initial_value">0.0</param>
             </state_interface>
             <state_interface name="velocity"/>
@@ -109,4 +136,7 @@
                 <param name="min">-1.57</param>
                 <param name="max">1.57</param>
+                <param name="p">100.0</param>
+                <param name="i">0.0</param>
+                <param name="d">5.0</param>
             </command_interface>
             <state_interface name="position">
@@ -120,7 +150,10 @@
                 <param name="min">-1.2217</param>
                 <param name="max">3.14</param>
+                <param name="p">150.0</param>
+                <param name="i">0.0</param>
+                <param name="d">10.0</param>
             </command_interface>
             <state_interface name="position">
-                <param name="initial_value">0.0</param>
+                <param name="initial_value">-0.7854</param>
             </state_interface>
             <state_interface name="velocity"/>
@@ -131,7 +164,10 @@
                 <param name="min">0.45</param>
                 <param name="max">2.3562</param>
+                <param name="p">50.0</param>
+                <param name="i">0.0</param>
+                <param name="d">2.0</param>
             </command_interface>
             <state_interface name="position">
-                <param name="initial_value">0.45</param>
+                <param name="initial_value">0.0</param>
             </state_interface>
             <state_interface name="velocity"/>
