Commit message: feat(hardware-layer-can): add CAN system support and update URDF control file

File: opendog_description/urdf/opendog_ros2_control.xacro (robot description, xacro)
@@ -175,79 +175,4 @@
       </joint>
     </ros2_control>
-    <!-- Définition des joints avec limites sécurisées -->
-    <!--
-    <joint name="FR_hip_joint" type="revolute">
-      <command_interface name="position"/>
-      <state_interface name="position"/>
-      <state_interface name="velocity"/>
-      <limit lower="0.515" upper="0.615" effort="100" velocity="100"/>
-    </joint>
-    <joint name="FL_hip_joint" type="revolute">
-      <command_interface name="position"/>
-      <state_interface name="position"/>
-      <state_interface name="velocity"/>
-      <limit lower="-0.045" upper="0.055" effort="100" velocity="100"/>
-    </joint>
-    <joint name="BR_hip_joint" type="revolute">
-      <command_interface name="position"/>
-      <state_interface name="position"/>
-      <state_interface name="velocity"/>
-      <limit lower="0.323" upper="0.423" effort="100" velocity="100"/>
-    </joint>
-    <joint name="BL_hip_joint" type="revolute">
-      <command_interface name="position"/>
-      <state_interface name="position"/>
-      <state_interface name="velocity"/>
-      <limit lower="0.166" upper="0.266" effort="100" velocity="100"/>
-    </joint>
-    <joint name="FR_uleg_joint" type="revolute">
-      <command_interface name="position"/>
-      <state_interface name="position"/>
-      <state_interface name="velocity"/>
-      <limit lower="-0.770" upper="-0.170" effort="100" velocity="100"/>
-    </joint>
-    <joint name="FL_uleg_joint" type="revolute">
-      <command_interface name="position"/>
-      <state_interface name="position"/>
-      <state_interface name="velocity"/>
-      <limit lower="-0.499" upper="0.101" effort="100" velocity="100"/>
-    </joint>
-    <joint name="BR_uleg_joint" type="revolute">
-      <command_interface name="position"/>
-      <state_interface name="position"/>
-      <state_interface name="velocity"/>
-      <limit lower="-0.150" upper="0.450" effort="100" velocity="100"/>
-    </joint>
-    <joint name="BL_uleg_joint" type="revolute">
-      <command_interface name="position"/>
-      <state_interface name="position"/>
-      <state_interface name="velocity"/>
-      <limit lower="0.166" upper="0.766" effort="100" velocity="100"/>
-    </joint>
-    <joint name="FR_lleg_joint" type="revolute">
-      <command_interface name="position"/>
-      <state_interface name="position"/>
-      <state_interface name="velocity"/>
-      <limit lower="-0.698" upper="3.839" effort="100" velocity="100"/>
-    </joint>
-    <joint name="FL_lleg_joint" type="revolute">
-      <command_interface name="position"/>
-      <state_interface name="position"/>
-      <state_interface name="velocity"/>
-      <limit lower="0.042" upper="0.642" effort="100" velocity="100"/>
-    </joint>
-    <joint name="BR_lleg_joint" type="revolute">
-      <command_interface name="position"/>
-      <state_interface name="position"/>
-      <state_interface name="velocity"/>
-      <limit lower="-0.611" upper="-0.011" effort="100" velocity="100"/>
-    </joint>
-    <joint name="BL_lleg_joint" type="revolute">
-      <command_interface name="position"/>
-      <state_interface name="position"/>
-      <state_interface name="velocity"/>
-      <limit lower="-0.538" upper="0.062" effort="100" velocity="100"/>
-    </joint>
-    -->
   </xacro:macro>
 </robot>
