Commit message: Address remaining hidden review comments on PR #31

File: opendog_description/urdf/opendog_stand_joints.xacro (robot description, xacro)
@@ -5,10 +5,10 @@
   <parent link="world"/>
   <child link="stand_link"/>
-  <origin xyz="0 0 0.1" rpy="0 0 0"/> <!-- Centre du cylindre à 0.5m -->
+  <origin xyz="0 0 0.1" rpy="0 0 0"/> <!-- Cylinder center at 0.5m -->
 </joint>
   <!-- Joint fixe entre stand et base_link -->
 <joint name="stand_to_base" type="fixed">
   <origin xyz="0 0 0.3" rpy="0 0 0"/>
-  <!-- Positionné au sommet du stand (z=0.5 + 0.5 = 1m) -->
+  <!-- Positioned at the top of the stand (z=0.5 + 0.5 = 1m) -->
   <parent link="stand_link"/>
   <child link="base_link"/>

File: opendog_description/urdf/opendog_stand_links.xacro (robot description, xacro)
@@ -1,5 +1,5 @@
 <?xml version="1.0" ?>
 <robot  xmlns:xacro="http://www.ros.org/wiki/xacro">
- <!-- Définition du lien du stand -->
+ <!-- Stand link definition -->
  <!-- World link -->
  <link name="world"/>
@@ -10,5 +10,5 @@
       <box size="0.5 0.5 0.2"/>
     </geometry>
-    <material name="green"> <!-- Changez le nom pour éviter les conflits -->
+    <material name="green"> <!-- Change the name to avoid conflicts -->
       <color rgba="0 0 0.8 1.0"/>
     </material>
@@ -25,5 +25,5 @@
   </inertial>
   </link>
-    <!-- Gazebo - rendre le stand statique pour éviter que le robot "tourne" dans la simulation -->
+    <!-- Gazebo - make the stand static so the robot doesn't "spin" in simulation -->
     <gazebo reference="stand_link">
       <static>true</static>
