Commit message: Add front/back test rigs, fix CAN activation retry/arbitration handling
- New front_test_* files (6-joint FL+FR rig)
- New back_test_* files (6-joint BL+BR rig, rebuilt from scratch)
- New back_test_legs_* files (4-joint legs-only rig, no hips)
- New fl_leg_test_*/fr_leg_test_* single-leg test rigs
- idle_and_clear_all_axes(): per-node retry with descending node-ID
  check order (CAN arbitration favors low IDs), widened stagger
- write(): round-robin gate on closed-loop retry to avoid all axes
  retrying in the same burst
- axis1 nodes given longer wait/more retries than axis0 (empirically
  needed more time to respond)

File: odrive_ros2_control_can/test/urdf/two_joints_test.urdf.xacro (robot description, xacro)
@@ -24,5 +24,5 @@
     </hardware>
     <joint name="motor_joint_0">
-      <param name="node_id">0</param>
+      <param name="node_id">6</param>
       <param name="axis">0</param>
       <param name="torque_constant">8.27</param>
@@ -35,5 +35,5 @@
     </joint>
     <joint name="motor_joint_1">
-      <param name="node_id">1</param>
+      <param name="node_id">7</param>
       <param name="axis">1</param>
       <param name="torque_constant">8.27</param>

File: opendog_hardware_layer_can/urdf/back_test_legs_ros2_control.xacro (robot description, xacro)
@@ -1,5 +1,5 @@
 <?xml version="1.0"?>
 <robot xmlns:xacro="http://www.ros.org/wiki/xacro">
-  <xacro:macro name="br_leg_test_ros2_control" params="name">
+  <xacro:macro name="back_test_legs_ros2_control" params="name">
     <ros2_control name="${name}" type="system">
       <hardware>
@@ -7,4 +7,26 @@
         <param name="can_interface">can0</param>
       </hardware>
+      <joint name="BL_uleg_joint">
+        <param name="node_id">4</param>
+        <param name="axis">0</param>
+        <param name="torque_constant">8.27</param>
+        <param name="gear_ratio">10.0</param>
+        <param name="enable_watchdog">false</param>
+        <param name="watchdog_timeout">0.1</param>
+        <command_interface name="position"/>
+        <state_interface name="position"/>
+        <state_interface name="velocity"/>
+      </joint>
+      <joint name="BL_lleg_joint">
+        <param name="node_id">5</param>
+        <param name="axis">1</param>
+        <param name="torque_constant">8.23</param>
+        <param name="gear_ratio">10.0</param>
+        <param name="enable_watchdog">false</param>
+        <param name="watchdog_timeout">0.1</param>
+        <command_interface name="position"/>
+        <state_interface name="position"/>
+        <state_interface name="velocity"/>
+      </joint>
       <joint name="BR_uleg_joint">
         <param name="node_id">10</param>
@@ -13,5 +35,5 @@
         <param name="gear_ratio">-10.0</param>
         <param name="zero_offset">0.62836</param>
-        <param name="enable_watchdog">true</param>
+        <param name="enable_watchdog">false</param>
         <param name="watchdog_timeout">0.1</param>
         <command_interface name="position"/>
@@ -22,7 +44,7 @@
         <param name="node_id">11</param>
         <param name="axis">1</param>
-        <param name="torque_constant">8.27</param>
+        <param name="torque_constant">8.23</param>
         <param name="gear_ratio">-10.0</param>
-        <param name="enable_watchdog">true</param>
+        <param name="enable_watchdog">false</param>
         <param name="watchdog_timeout">0.1</param>
         <command_interface name="position"/>

File: opendog_hardware_layer_can/urdf/fl_leg_test_ros2_control.xacro (robot description, xacro)
@@ -1,5 +1,5 @@
 <?xml version="1.0"?>
 <robot xmlns:xacro="http://www.ros.org/wiki/xacro">
-  <xacro:macro name="bl_leg_test_ros2_control" params="name">
+  <xacro:macro name="fl_leg_test_ros2_control" params="name">
     <ros2_control name="${name}" type="system">
       <hardware>
@@ -7,9 +7,10 @@
         <param name="can_interface">can0</param>
       </hardware>
-      <joint name="BL_uleg_joint">
-        <param name="node_id">4</param>
+      <joint name="FL_uleg_joint">
+        <param name="node_id">0</param>
         <param name="axis">0</param>
         <param name="torque_constant">8.27</param>
-        <param name="gear_ratio">10.0</param>
+        <param name="gear_ratio">-10.0</param>
+        <param name="zero_offset">1.199583</param>
         <param name="enable_watchdog">true</param>
         <param name="watchdog_timeout">0.1</param>
@@ -18,6 +19,6 @@
         <state_interface name="velocity"/>
       </joint>
-      <joint name="BL_lleg_joint">
-        <param name="node_id">5</param>
+      <joint name="FL_lleg_joint">
+        <param name="node_id">1</param>
         <param name="axis">1</param>
         <param name="torque_constant">8.27</param>

File: opendog_hardware_layer_can/urdf/fr_leg_test_ros2_control.xacro (robot description, xacro)
@@ -1,5 +1,5 @@
 <?xml version="1.0"?>
 <robot xmlns:xacro="http://www.ros.org/wiki/xacro">
-  <xacro:macro name="bl_leg_test_ros2_control" params="name">
+  <xacro:macro name="fr_leg_test_ros2_control" params="name">
     <ros2_control name="${name}" type="system">
       <hardware>
@@ -7,6 +7,6 @@
         <param name="can_interface">can0</param>
       </hardware>
-      <joint name="BL_uleg_joint">
-        <param name="node_id">4</param>
+      <joint name="FR_uleg_joint">
+        <param name="node_id">0</param>
         <param name="axis">0</param>
         <param name="torque_constant">8.27</param>
@@ -18,6 +18,6 @@
         <state_interface name="velocity"/>
       </joint>
-      <joint name="BL_lleg_joint">
-        <param name="node_id">5</param>
+      <joint name="FR_lleg_joint">
+        <param name="node_id">1</param>
         <param name="axis">1</param>
         <param name="torque_constant">8.27</param>
